Commit message: Imported upstream version '0.6.4' of 'upstream'

File: raw_description/urdf/base_long/base.urdf.xacro (robot description, xacro)
@@ -80,5 +80,5 @@
         <origin xyz="0 0 0.209" rpy="0 0 0" />
         <geometry>
-          <mesh filename="package://raw_description/meshes/base/raw_base_short.stl"/>
+          <mesh filename="package://raw_description/meshes/base/raw_base_long.stl"/>
           <!--box size="1.04 0.58 0.31" /-->
         </geometry>
