Commit message: Rebase from 'release/indigo/raw_description'

File: urdf/base_short/base.urdf.xacro (robot description, xacro)
@@ -3,12 +3,10 @@
   <xacro:include filename="$(find cob_description)/urdf/common.xacro"/>
   <xacro:include filename="$(find raw_description)/urdf/base_short/base.gazebo.xacro" />
-  <xacro:include filename="$(find raw_description)/urdf/base_short/base.transmission.xacro" />
+  <!-- drive_wheel module -->
+  <xacro:include filename="$(find cob_description)/urdf/drive_wheel/drive_wheel.urdf.xacro" />
   <!-- sensors -->
-  <xacro:include filename="$(find cob_description)/urdf/sensors/kinect.urdf.xacro" />
   <xacro:include filename="$(find cob_description)/urdf/sensors/sick_s300_laser.urdf.xacro"/>
-  <!-- DATA SOURCES -->
-  <!-- all link offsets, CG, limits are obtained from Function Engineering spreadsheet 090224_link_data.xls unless stated otherwise -->
-  <!-- all link geometry sizes are obtained from Function provided CAD model unless stated otherwise -->
-  <!-- all simplified collision geometry are hand approximated from CAD model, sometimes from respective bounding boxes -->
+  <xacro:include filename="$(find cob_description)/urdf/sensors/kinect.urdf.xacro"/>
+  <!-- properties -->
   <property name="caster_offset_x" value="0.228" />  <!--modify here-->
   <property name="caster_offset_y_bl" value="0.134" />
@@ -17,113 +15,12 @@
   <property name="caster_offset_y_fr" value="-0.134" />
   <property name="caster_offset_z" value="0.09" />
-  <property name="battery_offset_x_f" value="0.0" />
-  <property name="battery_offset_y_f" value="-0.008" />
+  <property name="battery_offset_x" value="0.0" />
+  <property name="battery_offset_y" value="-0.008" />
   <property name="battery_offset_z" value="0.065" />
-  <property name="caster_wheel_offset_y" value="0 " />
-  <property name="wheel_length" value="0.034" />
-  <property name="wheel_radius" value="0.074792" />   <!-- This is the 'effective' wheel radius. Wheel radius for uncompressed wheel is 0.079.  mp 20080801 -->
-  <!--property name="wheel_radius" value="0.08" /-->
-  <!--property name="base_cg_x" value="0" />
-  <property name="base_cg_y" value="0.0" />
-  <property name="base_cg_z" value="0" /!-->
   <property name="base_mass" value="43.1" />
-  <property name="battery_mass" value="40" />  <!--to be checked out-->
-  <property name="caster_mass" value="5.9" />
-  <!-- simplified box collision geometry for battery -->
+  <property name="battery_mass" value="40" />
   <property name="battery_size_x" value="0.5" />
   <property name="battery_size_y" value="0.148" />
   <property name="battery_size_z" value="0.26" />
-  <property name="base_laser_x" value="0.32501" />
-  <property name="base_laser_y_back" value="0.232" />
-  <property name="base_laser_y_front" value="0.232" />
-  <property name="base_laser_z" value="0.178" />
-  <!--                                                      -->
-  <!--           wheel                                      -->
-  <!--                                                      -->
-  <xacro:macro name="cob_wheel" params="suffix parent reflect">
-    <joint name="${parent}_${suffix}_wheel_joint" type="continuous">
-      <axis xyz="0 1 0" />
-      <limit effort="100" velocity="100"/> <!-- alpha tested effort and velocity limits -->
-      <safety_controller  k_velocity="10" />
-      <dynamics damping="0.0" friction="0.0" />
-      <origin xyz="0 ${reflect*caster_wheel_offset_y} 0" rpy="0 0 0" />
-      <parent link="${parent}_rotation_link"/>
-      <child link="${parent}_${suffix}_wheel_link"/>
-    </joint>
-    <link name="${parent}_${suffix}_wheel_link">
-      <inertial>
-        <mass value="0.44036" />
-        <origin xyz="0 0 0" />
-        <inertia  ixx="0.012411765597" ixy="-0.000711733678" ixz="0.00050272983"
-                  iyy="0.015218160428" iyz="-0.000004273467" izz="0.011763977943" />
-      </inertial>
-      <visual>
-        <origin xyz="0 0 0" rpy="0 0 0" />
-        <geometry>
-          <!--cylinder radius="${wheel_radius}" length="${wheel_length}" /-->
-          <mesh filename="package://raw_description/meshes/base/raw_wheel.dae"/>
-        </geometry>
-      </visual>
-      <collision>
-        <origin xyz="0 0 0" rpy="0 0 0" /> <!-- rotation because cyl. geom primitive has symmetry axis in +x direction -->
-        <geometry>
-          <!--cylinder radius="${wheel_radius}" length="${wheel_length}" /-->
-          <sphere radius="${wheel_radius}"/>
-          <!--mesh filename="package://raw_description/meshes/base/raw_wheel.stl"/-->
-        </geometry>
-      </collision>
-    </link>
-    <!-- extensions -->
-    <xacro:cob_wheel_gazebo parent="${parent}" suffix="${suffix}" />
-    <xacro:cob_wheel_transmission parent="${parent}" suffix="${suffix}" reflect="${reflect}" />
-  </xacro:macro>
-  <!-- Macro for Caster hub only -->
-  <xacro:macro name="cob_caster_hub" params="suffix parent *origin ref_position" >
-    <joint name="${suffix}_rotation_joint" type="continuous">
-      <axis xyz="0 0 1" />
-      <limit effort="100" velocity="100"/> <!-- alpha tested velocity and effort limits -->
-      <safety_controller  k_velocity="10" />
-      <calibration rising="${ref_position}"/>
-      <dynamics damping="0.0" friction="0.0" />
-      <insert_block name="origin" />
-      <parent link="${parent}"/>
-      <child link="${suffix}_rotation_link" />
-    </joint>
-    <link name="${suffix}_rotation_link">
-      <inertial>
-        <mass value="${caster_mass}"/>
-        <origin xyz="0 0 0" />
-        <inertia  ixx="0.04" ixy="-0.0007" ixz="0.0"
-                  iyy="0.02" iyz="-0.000004" izz="0.05" />
-      </inertial>
-      <visual>
-        <origin xyz="0 0 0" rpy="0 0 0" />
-        <geometry>
-          <mesh filename="package://raw_description/meshes/base/raw_caster.stl"/>
-          <!--box size="0.001 0.001 0.001" /-->
-        </geometry>
-        <material name="IPA/LightGrey" />
-      </visual>
-      <collision>
-        <origin xyz="0 0 0" rpy="0 0 0" />
-        <geometry>
-          <box size="0.001 0.001 0.001" />
-        </geometry>
-      </collision>
-    </link>
-    <!-- extensions -->
-    <xacro:cob_caster_transmission suffix="${suffix}" />
-  </xacro:macro>
-  <xacro:macro name="cob_caster" params="suffix parent *origin ref_position">
-    <xacro:cob_caster_hub parent="${parent}" suffix="${suffix}_caster"
-                             ref_position="${ref_position}" >
-      <insert_block name="origin" />
-    </xacro:cob_caster_hub>
-    <!-- wheel macros -->
-    <!--xacro:cob_wheel parent="${suffix}_caster" suffix="l" reflect="1" /--> <!--### modified by jie ###-->
-    <xacro:cob_wheel parent="${suffix}_caster" suffix="r" reflect="-1" />
-    <!-- extensions -->
-    <xacro:cob_caster_gazebo suffix="${suffix}" />
-  </xacro:macro>
   <!-- battery macros-->
   <xacro:macro name="cob_batteries" params="name parent *origin ">
@@ -135,6 +32,6 @@
     <link name="${name}_battery">
       <inertial>
+        <origin xyz="0 0 0" />
         <mass value="${battery_mass}" />
-        <origin xyz="0 0 0" />
         <inertia ixx="0.01" ixy="0.0" ixz="0.0"
                  iyy="0.01" iyz="0.0" izz="0.01" />
@@ -146,5 +43,5 @@
         </geometry>
         <material name="Gazebo/Black" />
-       </visual>
+      </visual>
       <collision>
         <origin xyz="0 0.075 0" rpy="0 0 0"/> <!-- TODO: Change the origin of the stl, so that collision model doesn't need to be translated  -->
@@ -156,12 +53,17 @@
     </link>
     <!-- extensions -->
-    <xacro:cob_batteries_gazebo name="${name}" />
+    <xacro:batteries_gazebo name="${name}" />
   </xacro:macro>
-  <!-- The xacro macro xacro:cob_base contains: base, casters and wheels -->
   <xacro:macro name="raw_base" params="name">
+    <link name="${name}_footprint"/>
+    <joint name="${name}_footprint_joint" type="fixed">
+      <origin xyz="0 0 0" rpy="0 0 0" />
+      <parent link="${name}_footprint"/>
+      <child link="${name}_link" />
+    </joint>
     <link name="${name}_link">
       <inertial>
+        <origin xyz="0 0 0" />
         <mass value="${base_mass}" />
-        <origin xyz="0 0 0" />
         <inertia ixx="9.64" ixy="-0.02" ixz="0.44"
                  iyy="11.33" iyz="-0.007" izz="3.07" />
@@ -176,49 +78,40 @@
         <origin xyz="0 0 0.209" rpy="0 0 0" />
         <geometry>
-          <!--box size="0.758 0.573 0.096"/--> <!-- Laserscan measures inside this box -->
           <mesh filename="package://raw_description/meshes/base/raw_base_short.stl"/>
+          <!--box size="0.758 0.573 0.096"/-->
         </geometry>
       </collision>
     </link>
-    <!-- base_footprint is a fictitious link(frame) that is on the ground right below base_link origin,
-         navigation stack dedpends on this frame -->
-    <link name="${name}_footprint"/>
-    <joint name="${name}_footprint_joint" type="fixed">
-      <origin xyz="0 0 0" rpy="0 0 0" />
-      <child link="${name}_link" />
-      <parent link="${name}_footprint"/>
-    </joint>
-    <!--modify here for test: front,base and top lasers -->
+    <!-- arrangement of the four drive_wheel modules -->
+    <xacro:drive_wheel parent="${name}_link" suffix="fl" >
+      <origin xyz="${caster_offset_x} ${caster_offset_y_fl} ${caster_offset_z}" rpy="0 0 0" />
+    </xacro:drive_wheel>
+    <xacro:drive_wheel parent="${name}_link" suffix="fr" >
+      <origin xyz="${caster_offset_x} ${caster_offset_y_fr} ${caster_offset_z}" rpy="0 0 0" />
+    </xacro:drive_wheel>
+    <xacro:drive_wheel parent="${name}_link" suffix="bl" >
+      <origin xyz="${-caster_offset_x} ${caster_offset_y_bl} ${caster_offset_z}" rpy=" 0 0 0" />
+    </xacro:drive_wheel>
+    <xacro:drive_wheel parent="${name}_link" suffix="br"  >
+      <origin xyz="${-caster_offset_x} ${caster_offset_y_br} ${caster_offset_z}" rpy="0 0 0" />
+    </xacro:drive_wheel>
     <!-- base laser front -->
     <xacro:sick_s300_laser_v0 name="${name}_laser_front" parent="${name}" ros_topic="scan_front_raw" update_rate="10" min_angle="-2.3562" max_angle="2.3562" >
-      <origin xyz="${base_laser_x} ${-base_laser_y_front} ${base_laser_z}" rpy="${M_PI} 0 ${-M_PI/4}" />
+      <origin xyz="${laser_front_x} ${laser_front_y} ${laser_front_z}" rpy="${laser_front_roll} ${laser_front_pitch} ${laser_front_yaw}" />
     </xacro:sick_s300_laser_v0>
     <!-- base laser rear -->
     <xacro:sick_s300_laser_v0 name="${name}_laser_rear" parent="${name}" ros_topic="scan_rear_raw" update_rate="10" min_angle="-2.3562" max_angle="2.3562" >
-      <origin xyz="${-base_laser_x} ${base_laser_y_back} ${base_laser_z}" rpy="${M_PI} 0 ${-5*M_PI/4}" />
+      <origin xyz="${laser_front_x} ${laser_front_y} ${laser_front_z}" rpy="${laser_front_roll} ${laser_front_pitch} ${laser_front_yaw}" />
     </xacro:sick_s300_laser_v0>
+    <!-- cam3d -->
+    <!--xacro:cob_kinect_v0 name="${name}_cam3d" ros_topic="cam3d" parent="${name}_link">
+      <origin xyz="0.51 0.12 0.27" rpy="-${M_PI/2} 0 -${M_PI/2}" />
+    </xacro:cob_kinect_v0-->
     <!-- battery-->
     <xacro:cob_batteries name="${name}_battery" parent="${name}_link">
-      <origin xyz="${-battery_offset_x_f} ${battery_offset_y_f} ${battery_offset_z}" rpy="${M_PI/2} 0 ${-M_PI/2}" />
+      <origin xyz="${-battery_offset_x} ${battery_offset_y} ${battery_offset_z}" rpy="${M_PI/2} 0 ${-M_PI/2}" />
     </xacro:cob_batteries>
-    <!-- all four caster macros -->
-    <xacro:cob_caster suffix="fl" parent="${name}_link" ref_position="${cal_caster_fl - M_PI/4}" >
-      <origin xyz="${caster_offset_x} ${caster_offset_y_fl} ${caster_offset_z}" rpy="0 0 0" />
-    </xacro:cob_caster>
-    <xacro:cob_caster suffix="fr" parent="${name}_link" ref_position="${cal_caster_fr - M_PI/4}" >
-      <origin xyz="${caster_offset_x} ${caster_offset_y_fr} ${caster_offset_z}" rpy="0 0 0" />
-    </xacro:cob_caster>
-    <xacro:cob_caster suffix="bl" parent="${name}_link" ref_position="${cal_caster_bl - M_PI / 4 + M_PI}" >
-      <origin xyz="${-caster_offset_x} ${caster_offset_y_bl} ${caster_offset_z}" rpy=" 0 0 0" />
-    </xacro:cob_caster>
-    <xacro:cob_caster suffix="br" parent="${name}_link" ref_position="${cal_caster_br - M_PI / 4 + M_PI}"  >
-      <origin xyz="${-caster_offset_x} ${caster_offset_y_br} ${caster_offset_z}" rpy="0 0 0" />
-    </xacro:cob_caster>
-   <!-- cam3d -->
-   <!--xacro:cob_kinect_v0 name="${name}_cam3d" ros_topic="cam3d" parent="${name}_link">
-      <origin xyz="0.51 0.12 0.27" rpy="-${M_PI/2} 0 -${M_PI/2}" />
-   </xacro:cob_kinect_v0-->
     <!-- gazebo extensions -->
-    <xacro:cob_base_gazebo name="${name}" />
+    <xacro:base_gazebo name="${name}" />
   </xacro:macro>
 </robot>

File: urdf/torso/torso.urdf.xacro (robot description, xacro)
@@ -37,5 +37,4 @@
       <axis xyz="0 0 -1.0" />
       <dynamics damping="25.0" friction="10.0"/>
-      <calibration rising="${torso_pan_ref}"/>
       <limit effort="41.4" lower="-6.2831" upper="6.2831" velocity="0.5"/>
     </joint>
@@ -67,5 +66,4 @@
       <axis xyz="0 1.0 0" />
       <dynamics damping="0.1" />
-      <calibration rising="${torso_tilt_ref}"/>
       <limit effort="100" lower="-3.2" upper="1.57" velocity="1.4"/>
     </joint>
