Commit message: Imported upstream version '0.6.5' of 'upstream'

File: cob_description/urdf/cob3_base/base.urdf.xacro (robot description, xacro)
@@ -54,13 +54,13 @@
     </xacro:drive_wheel>
     <!-- base laser front -->
-    <xacro:sick_s300_laser_v0 name="${name}_laser_front" parent="${name}" ros_topic="scan_front_raw" update_rate="10" min_angle="-2.3562" max_angle="2.3562" >
+    <xacro:sick_s300_laser_v0 name="${name}_laser_front" parent="${name}">
       <origin xyz="${laser_front_x} ${laser_front_y} ${laser_front_z}" rpy="${laser_front_roll} ${laser_front_pitch} ${laser_front_yaw}" />
     </xacro:sick_s300_laser_v0>
     <!-- base laser rear -->
-    <xacro:sick_s300_laser_v0 name="${name}_laser_rear" parent="${name}" ros_topic="scan_rear_raw" update_rate="10" min_angle="-2.3562" max_angle="2.3562" >
+    <xacro:sick_s300_laser_v0 name="${name}_laser_rear" parent="${name}">
       <origin xyz="${laser_rear_x} ${laser_rear_y} ${laser_rear_z}" rpy="${laser_rear_roll} ${laser_rear_pitch} ${laser_rear_yaw}" />
     </xacro:sick_s300_laser_v0>
     <!-- base laser top -->
-    <xacro:hokuyo_lx30_laser_v0 name="${name}_laser_top" parent="${name}" ros_topic="scan_top_raw" update_rate="10" min_angle="-2.3562" max_angle="2.3562" >
+    <xacro:hokuyo_lx30_laser_v0 name="${name}_laser_top" parent="${name}">
       <origin xyz="${laser_top_x} ${laser_top_y} ${laser_top_z}" rpy="${laser_top_roll} ${laser_top_pitch} ${laser_top_yaw}" />
     </xacro:hokuyo_lx30_laser_v0>

File: cob_description/urdf/cob4_base/base.urdf.xacro (robot description, xacro)
@@ -64,11 +64,11 @@
     </xacro:unless>
     <!-- sensors -->
-    <xacro:sick_s300_laser_v0 name="${name}_laser_front" parent="${name}" ros_topic="scan_front_raw" update_rate="12" min_angle="-2.094" max_angle="2.094" >
+    <xacro:sick_s300_laser_v0 name="${name}_laser_front" parent="${name}">
       <origin xyz="${laser_front_x} ${laser_front_y} ${laser_front_z}" rpy="${laser_front_roll} ${laser_front_pitch} ${laser_front_yaw}" />
     </xacro:sick_s300_laser_v0>
-    <xacro:sick_s300_laser_v0 name="${name}_laser_left" parent="${name}" ros_topic="scan_left_raw" update_rate="12" min_angle="-2.094" max_angle="2.094" >
+    <xacro:sick_s300_laser_v0 name="${name}_laser_left" parent="${name}">
       <origin xyz="${laser_left_x} ${laser_left_y} ${laser_left_z}" rpy="${laser_left_roll} ${laser_left_pitch} ${laser_left_yaw}" />
     </xacro:sick_s300_laser_v0>
-    <xacro:sick_s300_laser_v0 name="${name}_laser_right" parent="${name}" ros_topic="scan_right_raw" update_rate="12" min_angle="-2.094" max_angle="2.094" >
+    <xacro:sick_s300_laser_v0 name="${name}_laser_right" parent="${name}">
       <origin xyz="${laser_right_x} ${laser_right_y} ${laser_right_z}" rpy="${laser_right_roll} ${laser_right_pitch} ${laser_right_yaw}" />
     </xacro:sick_s300_laser_v0>

File: cob_description/urdf/cob4_torso/torso_2dof.urdf.xacro (robot description, xacro)
@@ -8,6 +8,6 @@
     <joint name="${name}_base_joint" type="fixed">
       <insert_block name="origin" />
+      <parent link="${parent}"/>
       <child link="${name}_base_link" />
-      <parent link="${parent}"/>
     </joint>
     <link name="${name}_base_link">
@@ -18,9 +18,21 @@
       </xacro:cylinder_inertial>
 -->
+      <visual>
+        <origin xyz="0 0 0" rpy="0 0 0" />
+        <geometry>
+          <box size="0.001 0.001 0.001" />
+        </geometry>
+      </visual>
+      <collision>
+        <origin xyz="0 0 0" rpy="0 0 0" />
+        <geometry>
+          <box size="0.001 0.001 0.001" />
+        </geometry>
+      </collision>
     </link>
     <joint name="${name}_1_joint" type="fixed">
       <origin xyz="0 0 0.04642" rpy="0 0 0"/>
+      <parent link="${name}_base_link"/>
       <child link="${name}_1_link" />
-      <parent link="${name}_base_link"/>
     </joint>
     <link name="${name}_1_link">
@@ -31,7 +43,19 @@
       </xacro:hollow_spherical_cap_inertial>
 -->
+      <visual>
+        <origin xyz="0 0 0" rpy="0 0 0" />
+        <geometry>
+          <box size="0.001 0.001 0.001" />
+        </geometry>
+      </visual>
+      <collision>
+        <origin xyz="0 0 0" rpy="0 0 0" />
+        <geometry>
+          <box size="0.001 0.001 0.001" />
+        </geometry>
+      </collision>
     </link>
     <joint name="${name}_2_joint" type="revolute">
-      <origin xyz="0 -0.14734 0.07547" rpy="-0.5236 0 0" />
+      <origin xyz="0 0.14734 0.07547" rpy="0.5236 0 0" />
       <parent link="${name}_1_link"/>
       <child link="${name}_2_link" />
@@ -46,7 +70,19 @@
       </xacro:spherical_cap_inertial>
 -->
+      <visual>
+        <origin xyz="0 0 0" rpy="0 0 0" />
+        <geometry>
+          <box size="0.001 0.001 0.001" />
+        </geometry>
+      </visual>
+      <collision>
+        <origin xyz="0 0 0" rpy="0 0 0" />
+        <geometry>
+          <box size="0.001 0.001 0.001" />
+        </geometry>
+      </collision>
     </link>
     <joint name="${name}_3_joint" type="revolute">
-      <origin xyz="0 0.09228 0.13477" rpy="0.5236 0 0" />
+      <origin xyz="0 -0.09228 0.13477" rpy="-0.5236 0 0" />
       <parent link="${name}_2_link"/>
       <child link="${name}_3_link" />
@@ -79,5 +115,19 @@
       <child link="${name}_center_link" />
     </joint>
-    <link name="${name}_center_link"/>
+    <link name="${name}_center_link">
+      <xacro:default_inertial/>
+      <visual>
+        <origin xyz="0 0 0" rpy="0 0 0" />
+        <geometry>
+          <box size="0.001 0.001 0.001" />
+        </geometry>
+      </visual>
+      <collision>
+        <origin xyz="0 0 0" rpy="0 0 0" />
+        <geometry>
+          <box size="0.001 0.001 0.001" />
+        </geometry>
+      </collision>
+    </link>
     <!-- left camera -->
     <xacro:cob_kinect_v0 name="${name}_cam3d_left" ros_topic="torso_cam3d_left" parent="${name}_3_link">

File: cob_description/urdf/cob4_torso/torso_3dof.urdf.xacro (robot description, xacro)
@@ -8,6 +8,6 @@
     <joint name="${name}_base_joint" type="fixed">
       <insert_block name="origin" />
+      <parent link="${parent}"/>
       <child link="${name}_base_link" />
-      <parent link="${parent}"/>
     </joint>
     <link name="${name}_base_link">
@@ -59,5 +59,5 @@
     </link>
     <joint name="${name}_2_joint" type="revolute">
-      <origin xyz="0 -0.14734 0.07547" rpy="-0.5236 0 0" />
+      <origin xyz="0 0.14734 0.07547" rpy="0.5236 0 0" />
       <parent link="${name}_1_link"/>
       <child link="${name}_2_link" />
@@ -86,5 +86,5 @@
     </link>
     <joint name="${name}_3_joint" type="revolute">
-      <origin xyz="0 0.09228 0.13477" rpy="0.5236 0 0" />
+      <origin xyz="0 -0.09228 0.13477" rpy="-0.5236 0 0" />
       <parent link="${name}_2_link"/>
       <child link="${name}_3_link" />

File: cob_description/urdf/cob4_torso/torso_static.urdf.xacro (robot description, xacro)
@@ -8,6 +8,6 @@
     <joint name="${name}_base_joint" type="fixed">
       <insert_block name="origin" />
+      <parent link="${parent}"/>
       <child link="${name}_base_link" />
-      <parent link="${parent}"/>
     </joint>
     <link name="${name}_base_link">
@@ -57,5 +57,5 @@
     </link>
     <joint name="${name}_2_joint" type="fixed">
-      <origin xyz="0 -0.14734 0.07547" rpy="-0.5236 0 0" />
+      <origin xyz="0 0.14734 0.07547" rpy="0.5236 0 0" />
       <parent link="${name}_1_link"/>
       <child link="${name}_2_link" />
@@ -82,5 +82,5 @@
     </link>
     <joint name="${name}_3_joint" type="fixed">
-      <origin xyz="0 0.09228 0.13477" rpy="0.5236 0 0" />
+      <origin xyz="0 -0.09228 0.13477" rpy="-0.5236 0 0" />
       <parent link="${name}_2_link"/>
       <child link="${name}_3_link" />

File: cob_description/urdf/sensors/hokuyo_lx30_laser.gazebo.xacro (robot description, xacro)
@@ -1,9 +1,9 @@
 <?xml version="1.0"?>
 <robot xmlns:xacro="http://www.ros.org/wiki/xacro">
-  <xacro:macro name="hokuyo_lx30_laser_gazebo_v0" params="name ros_topic update_rate min_angle max_angle">
+  <xacro:macro name="hokuyo_lx30_laser_gazebo_v0" params="name">
     <gazebo reference="${name}_link">
       <sensor name="${name}" type="ray">
         <always_on>true</always_on>
-        <update_rate>${update_rate}</update_rate>
+        <update_rate>10.0</update_rate>
         <pose>0 0 0 0 0 0</pose>
         <visualize>false</visualize>
@@ -13,6 +13,6 @@
               <samples>640</samples>
               <resolution>1.0</resolution>
-              <min_angle>${min_angle}</min_angle>
-              <max_angle>${max_angle}</max_angle>
+              <min_angle>-2.3562</min_angle>
+              <max_angle>2.3562</max_angle>
             </horizontal>
           </scan>
@@ -29,5 +29,5 @@
         </ray>
         <plugin name="gazebo_ros_${name}_controller" filename="libgazebo_ros_laser.so">
-          <topicName>${ros_topic}</topicName>
+          <topicName>${name}/scan_raw</topicName>
           <frameName>${name}_link</frameName>
         </plugin>

File: cob_description/urdf/sensors/hokuyo_lx30_laser.urdf.xacro (robot description, xacro)
@@ -2,5 +2,5 @@
 <robot xmlns:xacro="http://www.ros.org/wiki/xacro">
   <xacro:include filename="$(find cob_description)/urdf/sensors/hokuyo_lx30_laser.gazebo.xacro" />
-  <xacro:macro name="hokuyo_lx30_laser_v0" params="name parent *origin ros_topic update_rate min_angle max_angle">
+  <xacro:macro name="hokuyo_lx30_laser_v0" params="name parent *origin">
     <joint name="${name}_joint" type="fixed">
       <axis xyz="0 1 0" />
@@ -11,5 +11,5 @@
     <link name="${name}_link" type="laser"/>
     <!-- gazebo extensions -->
-    <xacro:hokuyo_lx30_laser_gazebo_v0 name="${name}" ros_topic="${ros_topic}" update_rate="${update_rate}" min_angle="${min_angle}" max_angle="${max_angle}" />
+    <xacro:hokuyo_lx30_laser_gazebo_v0 name="${name}"/>
   </xacro:macro>
 </robot>

File: cob_description/urdf/sensors/sick_3dcs.gazebo.xacro (robot description, xacro)
@@ -1,19 +1,19 @@
 <?xml version="1.0"?>
-<root xmlns:xacro="http://www.ros.org/wiki/xacro">
-  <xacro:macro name="cob_kinect_gazebo_v0" params="name ros_topic">
+<robot xmlns:xacro="http://www.ros.org/wiki/xacro">
+  <xacro:macro name="sick_3dcs_gazebo" params="name ros_topic">
     <gazebo reference="${name}_frame">
       <sensor type="depth" name="${name}_frame_sensor">
         <always_on>true</always_on>
-        <update_rate>20.0</update_rate>
+        <update_rate>25.0</update_rate>
         <camera>
-          <horizontal_fov>${62.0*M_PI/180.0}</horizontal_fov>
+          <horizontal_fov>${74.0*M_PI/180.0}</horizontal_fov>
           <image>
             <format>R8G8B8</format>
-            <width>640</width>
-            <height>480</height>
+            <width>320</width>
+            <height>240</height>
           </image>
           <clip>
-            <near>0.1</near>
-            <far>100</far>
+            <near>0.15</near>
+            <far>1.0</far>
           </clip>
           <noise>
@@ -23,17 +23,12 @@
           </noise>
         </camera>
-        <plugin name="${name}_controller" filename="libgazebo_ros_openni_kinect.so">
-          <updateRate>20.0</updateRate>
+        <plugin name="${name}_frame_controller" filename="libgazebo_ros_openni_kinect.so">
+          <updateRate>25.0</updateRate>
           <cameraName>${ros_topic}</cameraName>
-          <frameName>${name}_link</frameName>
-          <imageTopicName>rgb/image_raw</imageTopicName>
+          <pointCloudTopicName>depth_registered/points</pointCloudTopicName>
           <cameraInfoTopicName>rgb/camera_info</cameraInfoTopicName>
-          <pointCloudTopicName>depth_registered/points</pointCloudTopicName>
-          <depthImageTopicName>depth_registered/image_raw</depthImageTopicName>
           <depthImageCameraInfoTopicName>depth_registered/camera_info</depthImageCameraInfoTopicName>
           <pointCloudCutoff>0.5</pointCloudCutoff>
           <pointCloudCutoffMax>5.0</pointCloudCutoffMax>
-          <baseline>0.2</baseline>
-          <hackBaseline>0.0</hackBaseline>
           <distortionK1>0.0</distortionK1>
           <distortionK2>0.0</distortionK2>
@@ -50,3 +45,3 @@
     </gazebo>
   </xacro:macro>
-</root>
+</robot>

File: cob_description/urdf/sensors/sick_s300_laser.gazebo.xacro (robot description, xacro)
@@ -1,9 +1,9 @@
 <?xml version="1.0"?>
 <robot xmlns:xacro="http://www.ros.org/wiki/xacro">
-  <xacro:macro name="sick_s300_laser_gazebo_v0" params="name ros_topic update_rate min_angle max_angle">
+  <xacro:macro name="sick_s300_laser_gazebo_v0" params="name">
     <gazebo reference="${name}_link">
       <sensor name="${name}" type="ray">
         <always_on>true</always_on>
-        <update_rate>${update_rate}</update_rate>
+        <update_rate>12.0</update_rate>
         <pose>0 0 0 0 0 0</pose>
         <visualize>false</visualize>
@@ -13,6 +13,6 @@
               <samples>541</samples>
               <resolution>1.0</resolution>
-              <min_angle>${min_angle}</min_angle>
-              <max_angle>${max_angle}</max_angle>
+              <min_angle>-2.3562</min_angle>
+              <max_angle>2.3562</max_angle>
             </horizontal>
           </scan>
@@ -29,5 +29,5 @@
         </ray>
         <plugin name="gazebo_ros_${name}_controller" filename="libgazebo_ros_laser.so">
-          <topicName>${ros_topic}</topicName>
+          <topicName>${name}/scan_raw</topicName>
           <frameName>${name}_link</frameName>
         </plugin>

File: cob_description/urdf/sensors/sick_s300_laser.urdf.xacro (robot description, xacro)
@@ -4,5 +4,5 @@
   <property name="cylinder_radius" value="0.05" />  <!--simple collision model for the laser -->
   <property name="cylinder_length" value="0.15" />
-  <xacro:macro name="sick_s300_laser_v0" params="name parent *origin ros_topic update_rate min_angle max_angle">
+  <xacro:macro name="sick_s300_laser_v0" params="name parent *origin">
     <joint name="${name}_joint" type="fixed">
       <axis xyz="0 1 0" />
@@ -31,5 +31,5 @@
     </link>
     <!-- gazebo extensions -->
-    <xacro:sick_s300_laser_gazebo_v0 name="${name}" ros_topic="${ros_topic}" update_rate="${update_rate}" min_angle="${min_angle}" max_angle="${max_angle}" />
+    <xacro:sick_s300_laser_gazebo_v0 name="${name}"/>
   </xacro:macro>
 </robot>

File: cob_description/urdf/sensors/softkinetic.gazebo.xacro (robot description, xacro)
@@ -26,10 +26,10 @@
           <updateRate>25.0</updateRate>
           <cameraName>${ros_topic}</cameraName>
+          <frameName>${name}_optical_frame</frameName>
           <imageTopicName>rgb/image_raw</imageTopicName>
-          <depthImageTopicName>depth/image_raw</depthImageTopicName>
+          <cameraInfoTopicName>rgb/camera_info</cameraInfoTopicName>
           <pointCloudTopicName>depth_registered/points</pointCloudTopicName>
-          <cameraInfoTopicName>rgb/camera_info</cameraInfoTopicName>
+          <depthImageTopicName>depth_registered/image_raw</depthImageTopicName>
           <depthImageCameraInfoTopicName>depth_registered/camera_info</depthImageCameraInfoTopicName>
-          <frameName>${name}_optical_frame</frameName>
           <pointCloudCutoff>0.5</pointCloudCutoff>
           <pointCloudCutoffMax>5.0</pointCloudCutoffMax>

File: raw_description/urdf/base_long/base.urdf.xacro (robot description, xacro)
@@ -99,9 +99,9 @@
     </xacro:drive_wheel>
     <!-- base laser front -->
-    <xacro:sick_s300_laser_v0 name="${name}_laser_front" parent="${name}" ros_topic="scan_front_raw" update_rate="10" min_angle="-2.3562" max_angle="2.3562" >
+    <xacro:sick_s300_laser_v0 name="${name}_laser_front" parent="${name}">
       <origin xyz="${laser_front_x} ${laser_front_y} ${laser_front_z}" rpy="${laser_front_roll} ${laser_front_pitch} ${laser_front_yaw}" />
     </xacro:sick_s300_laser_v0>
     <!-- base laser rear -->
-    <xacro:sick_s300_laser_v0 name="${name}_laser_rear" parent="${name}" ros_topic="scan_rear_raw" update_rate="10" min_angle="-2.3562" max_angle="2.3562" >
+    <xacro:sick_s300_laser_v0 name="${name}_laser_rear" parent="${name}">
       <origin xyz="${laser_rear_x} ${laser_rear_y} ${laser_rear_z}" rpy="${laser_rear_roll} ${laser_rear_pitch} ${laser_rear_yaw}" />
     </xacro:sick_s300_laser_v0>

File: raw_description/urdf/base_short/base.urdf.xacro (robot description, xacro)
@@ -97,10 +97,10 @@
     </xacro:drive_wheel>
     <!-- base laser front -->
-    <xacro:sick_s300_laser_v0 name="${name}_laser_front" parent="${name}" ros_topic="scan_front_raw" update_rate="10" min_angle="-2.3562" max_angle="2.3562" >
+    <xacro:sick_s300_laser_v0 name="${name}_laser_front" parent="${name}">
       <origin xyz="${laser_front_x} ${laser_front_y} ${laser_front_z}" rpy="${laser_front_roll} ${laser_front_pitch} ${laser_front_yaw}" />
     </xacro:sick_s300_laser_v0>
     <!-- base laser rear -->
-    <xacro:sick_s300_laser_v0 name="${name}_laser_rear" parent="${name}" ros_topic="scan_rear_raw" update_rate="10" min_angle="-2.3562" max_angle="2.3562" >
-      <origin xyz="${laser_front_x} ${laser_front_y} ${laser_front_z}" rpy="${laser_front_roll} ${laser_front_pitch} ${laser_front_yaw}" />
+    <xacro:sick_s300_laser_v0 name="${name}_laser_rear" parent="${name}">
+      <origin xyz="${laser_rear_x} ${laser_rear_y} ${laser_rear_z}" rpy="${laser_rear_roll} ${laser_rear_pitch} ${laser_rear_yaw}" />
     </xacro:sick_s300_laser_v0>
     <!-- cam3d -->
