Commit message: Rebase from 'release/kinetic/raw_description'

File: urdf/vacuum_gripper/gripper.urdf.xacro (robot description, xacro)
@@ -32,7 +32,7 @@
         </visual>
         <collision>
-            <origin xyz="0 0 -0.048" rpy="0 0 0"/>
+            <origin xyz="0.01 0.04 -0.048" rpy="0 0 0"/>
             <geometry>
-                <mesh filename="package://raw_description/meshes/vacuum_gripper/vacuum_gripper.stl"/>
+                <box size="0.13 0.14 0.071"/>
             </geometry>
         </collision>
