Commit message: Rebase from 'release/kinetic/cob_description'

File: urdf/cob4_base/base.urdf.xacro (robot description, xacro)
@@ -8,6 +8,6 @@
   <xacro:property name="caster_offset_y" value="0.21515" />
   <xacro:property name="caster_offset_z" value="0.08" />
-  <xacro:property name="base_mass" value="50" />
-  <xacro:macro name="base" params="name use_old_joint_names">
+  <xacro:property name="base_mass" value="100" />
+  <xacro:macro name="base" params="name tricycle_mode:=false">
     <xacro:property name="drive_vel" value="19.95" />
     <xacro:property name="steer_vel" value="117.81" />
@@ -41,16 +41,16 @@
     </link>
     <!-- arrangement of the three drive_wheel modules -->
-    <xacro:if value="${use_old_joint_names}">
-      <xacro:drive_wheel parent="${name}_link" suffix="fl" >
+    <xacro:if value="${tricycle_mode}">
+      <xacro:drive_wheel parent="${name}_link" suffix="fl" passive="true" >
         <origin xyz="${caster_offset_x/2} ${caster_offset_y} ${caster_offset_z}" rpy="0 0 0" />
       </xacro:drive_wheel>
-      <xacro:drive_wheel parent="${name}_link" suffix="bl" >
+      <xacro:drive_wheel parent="${name}_link" suffix="b" >
         <origin xyz="${-caster_offset_x} 0.0 ${caster_offset_z}" rpy="0 0 0" />
       </xacro:drive_wheel>
-      <xacro:drive_wheel parent="${name}_link" suffix="br" >
+      <xacro:drive_wheel parent="${name}_link" suffix="fr" passive="true">
         <origin xyz="${caster_offset_x/2} ${-caster_offset_y} ${caster_offset_z}" rpy="0 0 0" />
       </xacro:drive_wheel>
     </xacro:if>
-    <xacro:unless value="${use_old_joint_names}">
+    <xacro:unless value="${tricycle_mode}">
       <xacro:drive_wheel parent="${name}_link" suffix="fl" >
         <origin xyz="${caster_offset_x/2} ${caster_offset_y} ${caster_offset_z}" rpy="0 0 0" />

File: urdf/cob4_gripper/gripper.urdf.xacro (robot description, xacro)
@@ -1,4 +1,5 @@
 <?xml version="1.0"?>
 <robot xmlns:xacro="http://www.ros.org/wiki/xacro">
+  <xacro:include filename="$(find cob_description)/urdf/common.xacro" />
   <xacro:include filename="$(find cob_description)/urdf/cob4_gripper/gripper.gazebo.xacro" />
   <xacro:include filename="$(find cob_description)/urdf/cob4_gripper/gripper.transmission.xacro" />

File: urdf/sensors/kinect.gazebo.xacro (robot description, xacro)
@@ -3,5 +3,5 @@
   <xacro:macro name="cob_kinect_gazebo_v0" params="name ros_topic
                                                    update_rate:=20 data_skip:=0 height:=480 width:=640">
-    <gazebo reference="${name}_frame">
+    <gazebo reference="${name}_link">
       <sensor type="depth" name="${name}_frame_sensor">
         <always_on>true</always_on>
@@ -10,5 +10,5 @@
           <horizontal_fov>${62.0*M_PI/180.0}</horizontal_fov>
           <image>
-            <format>R8G8B8</format>
+            <format>B8G8R8</format>
             <width>${height}</width>
             <height>${width}</height>
@@ -27,5 +27,5 @@
           <updateRate>${update_rate/(data_skip+1)}</updateRate>
           <cameraName>${ros_topic}</cameraName>
-          <frameName>${name}_link</frameName>
+          <frameName>${name}_optical_frame</frameName>
           <imageTopicName>rgb/image_raw</imageTopicName>
           <cameraInfoTopicName>rgb/camera_info</cameraInfoTopicName>

File: urdf/sensors/kinect.urdf.xacro (robot description, xacro)
@@ -9,7 +9,5 @@
     </joint>
     <link name="${name}_link">
-      <xacro:box_inertial x="0.18" y="0.035" z="0.05" mass="0.3">
-        <origin xyz="0 0 0" rpy="0 0 0" />
-      </xacro:box_inertial>
+      <xacro:default_inertial/>
       <visual>
         <origin xyz="0 0 -0.03" rpy="0 0 0" />
@@ -26,16 +24,10 @@
       </collision>
     </link>
-    <joint name="${name}_frame_joint" type="fixed">
-      <origin xyz="0 0 0" rpy="${M_PI/2} -${M_PI/2} 0" />
-      <parent link="${name}_link"/>
-      <child link="${name}_frame"/>
-    </joint>
-    <link name="${name}_frame"/>
     <!-- extensions -->
     <xacro:cob_kinect_gazebo_v0 name="${name}" ros_topic="${ros_topic}"
-    									       update_rate="${update_rate}"
-    									       data_skip="${data_skip}"
-									           height="${height}"
-									           width="${width}"/>
+                                               update_rate="${update_rate}"
+                                               data_skip="${data_skip}"
+                                               height="${height}"
+                                               width="${width}"/>
   </xacro:macro>
 </root>

File: urdf/sensors/prosilica.gazebo.xacro (robot description, xacro)
@@ -9,5 +9,5 @@
           <horizontal_fov>0.58</horizontal_fov>
           <image>
-            <format>R8G8B8</format>
+            <format>B8G8R8</format>
             <width>1360</width>
             <height>1024</height>

File: urdf/sensors/prosilica.urdf.xacro (robot description, xacro)
@@ -10,9 +10,5 @@
     </joint>
     <link name="${name}_link">
-      <inertial>
-        <mass value="0.01" />
-        <origin xyz="0 0 0" rpy="0 0 0"/>
-        <inertia ixx="0.0001" ixy="0" ixz="0" iyy="0.0001" iyz="0" izz="0.0001" />
-      </inertial>
+      <xacro:default_inertial/>
       <visual>
         <origin xyz="0 0 0" rpy="0 0 0" />

File: urdf/sensors/realsense_zr300.gazebo.xacro (robot description, xacro)
@@ -2,6 +2,6 @@
 <robot xmlns:xacro="http://www.ros.org/wiki/xacro">
   <!-- use default values of realsense_camera/r200_nodelet_rgbd -->
-  <xacro:macro name="realsense_gazebo" params="name ros_topic
-                                               depth_fps:=30.0 depth_height:=360 depth_width:=480
+  <xacro:macro name="realsense_zr300_gazebo" params="name ros_topic
+                                               depth_fps:=30.0 depth_height:=480 depth_width:=640
                                                color_fps:=30.0 color_height:=480 color_width:=640" >
     <gazebo reference="${name}_link">
@@ -17,6 +17,6 @@
           </image>
           <clip>
-            <near>0.15</near>
-            <far>1.0</far>
+            <near>0.55</near>
+            <far>2.8</far>
           </clip>
           <noise>
@@ -35,6 +35,6 @@
           <depthImageTopicName>depth/image_raw</depthImageTopicName>
           <depthImageCameraInfoTopicName>depth/camera_info</depthImageCameraInfoTopicName>
-          <pointCloudCutoff>0.5</pointCloudCutoff>
-          <pointCloudCutoffMax>5.0</pointCloudCutoffMax>
+          <pointCloudCutoff>0.55</pointCloudCutoff>
+          <pointCloudCutoffMax>2.8</pointCloudCutoffMax>
           <distortionK1>0.0</distortionK1>
           <distortionK2>0.0</distortionK2>
@@ -48,4 +48,5 @@
         </plugin>
       </sensor>
+      <!-- ToDo: add plugins for IMU, Fisheye, IR -->
       <material>IPA/LightGrey</material>
     </gazebo>

File: urdf/sensors/realsense_zr300.urdf.xacro (robot description, xacro)
@@ -1,6 +1,6 @@
 <?xml version="1.0"?>
 <robot xmlns:xacro="http://www.ros.org/wiki/xacro">
-  <xacro:include filename="$(find cob_description)/urdf/sensors/realsense.gazebo.xacro" />
-  <xacro:macro name="realsense" params="name parent ros_topic *origin">
+  <xacro:include filename="$(find cob_description)/urdf/sensors/realsense_zr300.gazebo.xacro" />
+  <xacro:macro name="realsense_zr300" params="name parent ros_topic *origin">
     <joint name="${name}_joint" type="fixed">
       <xacro:insert_block name="origin" />
@@ -13,5 +13,5 @@
        <origin xyz="0 0 0" rpy="0 0 0"/>
         <geometry>
-          <box size="0.002 0.002 0.002"/>
+          <box size="0.01 0.155 0.035"/>
         </geometry>
       </visual>
@@ -19,10 +19,10 @@
         <origin xyz="0.0 0.0 0.0" rpy="0 0 0"/>
         <geometry>
-          <box size="0.007 0.130 0.0118"/>
+          <box size="0.01 0.155 0.035"/>
         </geometry>
       </collision>
     </link>
     <!-- extensions -->
-    <xacro:realsense_gazebo name="${name}" ros_topic="${ros_topic}" />
+    <xacro:realsense_zr300_gazebo name="${name}" ros_topic="${ros_topic}" />
   </xacro:macro>
 </robot>

File: urdf/sensors/sick_3dcs.gazebo.xacro (robot description, xacro)
@@ -5,11 +5,11 @@
       <sensor type="depth" name="${name}_frame_sensor">
         <always_on>true</always_on>
-        <update_rate>25.0</update_rate>
+        <update_rate>30.0</update_rate>
         <camera>
           <horizontal_fov>${74.0*M_PI/180.0}</horizontal_fov>
           <image>
-            <format>R8G8B8</format>
-            <width>320</width>
-            <height>240</height>
+            <format>B8G8R8</format>
+            <width>176</width>
+            <height>144</height>
           </image>
           <clip>
@@ -23,10 +23,13 @@
           </noise>
         </camera>
-        <plugin name="${name}_frame_controller" filename="libgazebo_ros_openni_kinect.so">
+        <plugin name="${name}_frame_controller" filename="libgazebo_ros_depth_camera.so">
           <updateRate>25.0</updateRate>
           <cameraName>${ros_topic}</cameraName>
-          <pointCloudTopicName>depth_registered/points</pointCloudTopicName>
-          <cameraInfoTopicName>rgb/camera_info</cameraInfoTopicName>
-          <depthImageCameraInfoTopicName>depth_registered/camera_info</depthImageCameraInfoTopicName>
+          <frameName>${name}_optical_frame</frameName>
+          <!--imageTopicName>ir/image_raw</imageTopicName-->
+          <!--cameraInfoTopicName>ir/camera_info</cameraInfoTopicName-->
+          <pointCloudTopicName>depth/points</pointCloudTopicName>
+          <depthImageTopicName>depth/image</depthImageTopicName>
+          <depthImageCameraInfoTopicName>depth/camera_info</depthImageCameraInfoTopicName>
           <pointCloudCutoff>0.5</pointCloudCutoff>
           <pointCloudCutoffMax>5.0</pointCloudCutoffMax>

File: urdf/sensors/sick_3dcs.urdf.xacro (robot description, xacro)
@@ -9,4 +9,16 @@
     </joint>
     <link name="${name}_link"/>
+    <joint name="${name}_frame_joint" type="fixed">
+      <origin xyz="0 0 0" rpy="0 0 0" />
+      <parent link="${name}_link"/>
+      <child link="${name}_frame"/>
+    </joint>
+    <link name="${name}_frame"/>
+    <joint name="${name}_optical_frame_joint" type="fixed">
+      <origin xyz="0 0 0" rpy="-${M_PI/2} 0 -${M_PI/2}" />
+      <parent link="${name}_frame"/>
+      <child link="${name}_optical_frame"/>
+    </joint>
+    <link name="${name}_optical_frame"/>
     <!-- extensions -->
     <xacro:sick_3dcs_gazebo name="${name}" ros_topic="${ros_topic}" />

File: urdf/sensors/sick_s300_laser.urdf.xacro (robot description, xacro)
@@ -6,5 +6,4 @@
   <xacro:macro name="sick_s300_laser_v0" params="name parent *origin">
     <joint name="${name}_joint" type="fixed">
-      <axis xyz="0 1 0" />
       <xacro:insert_block name="origin" />
       <parent link="${parent}_link"/>

File: urdf/sensors/usb_cam.gazebo.xacro (robot description, xacro)
@@ -3,5 +3,5 @@
   <!-- at 2048x1536 3.6hz is maximum on hw -->
   <xacro:macro name="usb_cam_gazebo" params="name ros_topic update_rate:=3.5 height:=1536 width:=2048" >
-    <gazebo reference="${name}_frame">
+    <gazebo reference="${name}_link">
     <sensor type="camera" name="${name}">
       <update_rate>${update_rate}</update_rate>
@@ -9,5 +9,5 @@
         <horizontal_fov>${170.0*M_PI/180.0}</horizontal_fov>
         <image>
-          <format>R8G8B8</format>
+          <format>B8G8R8</format>
           <width>${width}</width>
           <height>${height}</height>
@@ -29,5 +29,5 @@
         <imageTopicName>image_raw</imageTopicName>
         <cameraInfoTopicName>camera_info</cameraInfoTopicName>
-        <frameName>${name}_link</frameName>
+        <frameName>${name}_optical_frame</frameName>
         <hackBaseline>0.07</hackBaseline>
         <distortionK1>0.0</distortionK1>

File: urdf/sensors/usb_cam.urdf.xacro (robot description, xacro)
@@ -9,9 +9,5 @@
     </joint>
     <link name="${name}_link">
-      <inertial>
-        <mass value="0.1" />
-        <origin xyz="0 0 0" />
-        <inertia ixx="0.003881243" ixy="0.0" ixz="0.0" iyy="0.000498940" iyz="0.0" izz="0.003879257" />
-      </inertial>
+      <xacro:default_inertial/>
       <visual>
        <origin xyz="0 0 0" rpy="0 0 0"/>
@@ -28,14 +24,20 @@
     </link>
     <joint name="${name}_frame_joint" type="fixed">
-      <origin xyz="0 0 0" rpy="${M_PI/2} -${M_PI/2} 0" />
+      <origin xyz="0 0 0" rpy="0 0 0" />
       <parent link="${name}_link"/>
       <child link="${name}_frame"/>
     </joint>
     <link name="${name}_frame"/>
+    <joint name="${name}_optical_frame_joint" type="fixed">
+      <origin xyz="0 0 0" rpy="-${M_PI/2} 0 -${M_PI/2}" />
+      <parent link="${name}_frame"/>
+      <child link="${name}_optical_frame"/>
+    </joint>
+    <link name="${name}_optical_frame"/>
     <!-- extensions -->
     <xacro:usb_cam_gazebo name="${name}" ros_topic="${ros_topic}"
-									     update_rate="${update_rate}"
-									     height="${height}"
-									     width="${width}"/>
+                                         update_rate="${update_rate}"
+                                         height="${height}"
+                                         width="${width}"/>
   </xacro:macro>
 </robot>
