Commit message: Imported upstream version '0.6.6' of 'upstream'

File: cob_description/urdf/cob4_head/head.urdf.xacro (robot description, xacro)
@@ -47,5 +47,5 @@
     </link>
     <joint name="${name}_2_joint" type="revolute">
-      <origin xyz="0 -0.07725 -0.00439" rpy="0.349 0 0" />
+      <origin xyz="0 -0.07725 0.00439" rpy="0.349 0 0" />
       <parent link="${name}_1_link"/>
       <child link="${name}_2_link" />

File: cob_description/urdf/cob4_sensorring/sensorring.urdf.xacro (robot description, xacro)
@@ -29,5 +29,5 @@
       <child link="${name}_link" />
       <axis xyz="0 0 1" />
-      <limit effort="100" lower="-6.2831" upper="6.2831" velocity="6.28"/>
+      <limit effort="100" lower="-6.2831" upper="6.2831" velocity="2.62"/>
     </joint>
     <link name="${name}_link">

File: cob_description/urdf/cob4_sensorring/sensorring_3dcs_asus.urdf.xacro (robot description, xacro)
@@ -4,4 +4,5 @@
   <xacro:include filename="$(find cob_description)/urdf/cob4_sensorring/sensorring.transmission.xacro" />
   <xacro:include filename="$(find cob_description)/urdf/sensors/sick_3dcs.urdf.xacro" />
+  <xacro:include filename="$(find cob_description)/urdf/sensors/kinect.urdf.xacro" />
   <xacro:macro name="sensorring" params="parent name *origin">
     <joint name="${name}_base_joint" type="fixed">
@@ -52,8 +53,11 @@
       </collision>
     </link>
-    <!-- left camera -->
-    <xacro:sick_3dcs name="${name}_cam3d" ros_topic="sensorring_cam3d" parent="${name}_link">
-      <origin xyz="${sensorring_cam3d_x} ${sensorring_cam3d_y} ${sensorring_cam3d_z}" rpy="${sensorring_cam3d_roll} ${sensorring_cam3d_pitch} ${sensorring_cam3d_yaw}" />
+    <!-- camera -->
+    <xacro:sick_3dcs name="${name}_cam3d_front" ros_topic="${name}_cam3d_front" parent="${name}_link">
+      <origin xyz="${sensorring_cam3d_front_x} ${sensorring_cam3d_front_y} ${sensorring_cam3d_front_z}" rpy="${sensorring_cam3d_front_roll} ${sensorring_cam3d_front_pitch} ${sensorring_cam3d_front_yaw}" />
     </xacro:sick_3dcs>
+    <xacro:cob_kinect_v0 name="${name}_cam3d_back" ros_topic="${name}_cam3d_back" parent="${name}_link">
+      <origin xyz="${sensorring_cam3d_back_x} ${sensorring_cam3d_back_y} ${sensorring_cam3d_back_z}" rpy="${sensorring_cam3d_back_roll} ${sensorring_cam3d_back_pitch} ${sensorring_cam3d_back_yaw}" />
+    </xacro:cob_kinect_v0>
     <!-- extensions -->
     <xacro:sensorring_gazebo name="${name}" />

File: cob_description/urdf/cob4_sensorring/sensorring_asus.urdf.xacro (robot description, xacro)
@@ -30,5 +30,5 @@
       <child link="${name}_link" />
       <axis xyz="0 0 1" />
-      <limit effort="100" lower="-6.2831" upper="6.2831" velocity="6.28"/>
+      <limit effort="100" lower="-6.2831" upper="6.2831" velocity="2.62"/>
     </joint>
     <link name="${name}_link">

File: cob_description/urdf/common.xacro (robot description, xacro)
@@ -2,4 +2,20 @@
 <robot xmlns:xacro="http://www.ros.org/wiki/xacro">
   <property name="M_PI" value="3.1415926535897931" />
+  <!-- geometry macros for modeling geometric primitives with according meshes -->
+  <xacro:macro name="sphere_geometry" params="radius">
+    <geometry>
+      <mesh filename="package://cob_description/meshes/unit_sphere.stl" scale="${radius} ${radius} ${radius}"/>
+    </geometry>
+  </xacro:macro>
+  <xacro:macro name="cylinder_geometry" params="radius length">
+    <geometry>
+      <mesh filename="package://cob_description/meshes/unit_cylinder.stl" scale="${radius} ${radius} ${length}"/>
+    </geometry>
+  </xacro:macro>
+  <xacro:macro name="box_geometry" params="x y z">
+    <geometry>
+      <mesh filename="package://cob_description/meshes/unit_box.stl" scale="${x} ${y} ${z}"/>
+    </geometry>
+  </xacro:macro>
   <!-- see https://secure.wikimedia.org/wikipedia/en/wiki/List_of_moment_of_inertia_tensors -->
   <xacro:macro name="sphere_inertial" params="radius mass *origin">

File: cob_description/urdf/sensors/softkinetic.urdf.xacro (robot description, xacro)
@@ -8,11 +8,5 @@
       <child link="${name}_link"/>
     </joint>
-    <link name="${name}_link"/>
-    <joint name="${name}_frame_joint" type="fixed">
-      <origin xyz="0 0 0" rpy="${-M_PI/2} ${-M_PI/2} 0" />
-      <parent link="${name}_link"/>
-      <child link="${name}_frame"/>
-    </joint>
-    <link name="${name}_frame">
+    <link name="${name}_link">
       <xacro:box_inertial x="0.105" y="0.03" z="0.023" mass="0.5">
         <origin xyz="0 0 0" rpy="0 0 0" />
@@ -31,10 +25,29 @@
       </collision>
     </link>
-    <joint name="${name}_optical_joint" type="fixed">
-      <origin xyz="0 0 0" rpy="${-M_PI/2} 0.0 ${-M_PI/2}" />
-      <parent link="${name}_frame"/>
-      <child link="${name}_optical_frame"/>
+    <!-- Add frames for RGB and depth optical axes -->
+    <joint name="${name}_rgb_joint" type="fixed">
+      <origin xyz="0.0 0.0125 0.0" rpy="${-M_PI/2} ${-M_PI/2} 0.0"/>
+      <parent link="${name}_link"/>
+      <child link="${name}_rgb_frame"/>
     </joint>
-    <link name="${name}_optical_frame"/>
+    <link name="${name}_rgb_frame"/>
+    <joint name="${name}_rgb_optical_joint" type="fixed">
+      <origin xyz="0.0 0.0 0.0" rpy="${-M_PI/2} 0.0 ${-M_PI/2}"/>
+      <parent link="${name}_rgb_frame"/>
+      <child link="${name}_rgb_optical_frame"/>
+    </joint>
+    <link name="${name}_rgb_optical_frame"/>
+    <joint name="${name}_depth_joint" type="fixed">
+      <origin xyz="0.0 -0.0125 0.0" rpy="${-M_PI/2} ${-M_PI/2} 0.0"/>
+      <parent link="${name}_link"/>
+      <child link="${name}_depth_frame"/>
+    </joint>
+    <link name="${name}_depth_frame"/>
+    <joint name="${name}_depth_optical_joint" type="fixed">
+      <origin xyz="0.0 0.0 0.0" rpy="${-M_PI/2} 0.0 ${-M_PI/2}"/>
+      <parent link="${name}_depth_frame"/>
+      <child link="${name}_depth_optical_frame"/>
+    </joint>
+    <link name="${name}_depth_optical_frame"/>
     <!-- extensions -->
     <xacro:softkinetic_gazebo name="${name}" ros_topic="${ros_topic}" />

File: raw_description/urdf/base_long/base.urdf.xacro (robot description, xacro)
@@ -21,5 +21,5 @@
   <property name="battery_offset_z" value="0.065" />
   <property name="base_mass" value="83.1" />
-  <property name="battery_mass" value="83.1" />
+  <property name="battery_mass" value="25.0" />
   <property name="battery_size_x" value="0.5" />
   <property name="battery_size_y" value="0.148" />
@@ -33,10 +33,7 @@
     </joint>
     <link name="${name}_battery">
-      <inertial>
-        <origin xyz="0 0 0" />
-        <mass value="1.0" />
-        <inertia ixx="0.01" ixy="0.0" ixz="0.0"
-                 iyy="0.01" iyz="0.0" izz="0.01" />
-      </inertial>
+      <xacro:box_inertial x="${battery_size_x}" y="${battery_size_y}" z="${battery_size_z}" mass="${battery_mass}">
+        <origin xyz="0 0 0" rpy="0 0 0" />
+      </xacro:box_inertial>
       <visual>
         <origin xyz="0 0 0" rpy="0 0 0"/>

Commit message: Imported upstream version '0.7.0' of 'upstream'

File: cob_description/urdf/cob4_head/head.urdf.xacro (robot description, xacro)
@@ -127,5 +127,5 @@
     <xacro:head_transmission name="${name}" dof1="${dof1}" dof2="${dof2}" dof3="${dof3}" />
     <!-- ros_control plugin -->
-    <xacro:if value="${(dof1 == 'true') or (dof2 == 'true') or (dof3 == 'true')}">
+    <xacro:if value="${(dof1 == True) or (dof2 == True) or (dof3 == True)}">
       <gazebo>
         <plugin name="ros_control" filename="libhwi_switch_gazebo_ros_control.so">

File: cob_description/urdf/cob4_torso/torso.urdf.xacro (robot description, xacro)
@@ -3,5 +3,5 @@
   <xacro:include filename="$(find cob_description)/urdf/cob4_torso/torso.gazebo.xacro" />
   <xacro:include filename="$(find cob_description)/urdf/cob4_torso/torso.transmission.xacro" />
-  <xacro:macro name="torso" params="parent name *origin dof1:=false dof2:=false dof3:=false">
+  <xacro:macro name="torso" params="parent name *origin dof1:=False dof2:=False dof3:=False">
     <joint name="${name}_base_joint" type="fixed">
       <xacro:insert_block name="origin" />
@@ -161,5 +161,5 @@
     <xacro:torso_transmission name="${name}" dof1="${dof1}" dof2="${dof2}" dof3="${dof3}" />
     <!-- ros_control plugin -->
-    <xacro:if value="${(dof1 == 'true') or (dof2 == 'true') or (dof3 == 'true')}">
+    <xacro:if value="${(dof1 == True) or (dof2 == True) or (dof3 == True)}">
       <gazebo>
         <plugin name="ros_control" filename="libhwi_switch_gazebo_ros_control.so">

File: cob_description/urdf/common.xacro (robot description, xacro)
@@ -84,7 +84,7 @@
       <type>transmission_interface/SimpleTransmission</type>
       <joint name="${jname}_joint">
-        <hardwareInterface>PositionJointInterface</hardwareInterface>
-        <hardwareInterface>VelocityJointInterface</hardwareInterface>
-        <!--hardwareInterface>EffortJointInterface</hardwareInterface-->
+        <hardwareInterface>hardware_interface/PositionJointInterface</hardwareInterface>
+        <hardwareInterface>hardware_interface/VelocityJointInterface</hardwareInterface>
+        <!--hardwareInterface>hardware_interface/EffortJointInterface</hardwareInterface-->
       </joint>
       <actuator name="${jname}_motor">
