Commit message: Imported upstream version '0.6.7' of 'upstream'

File: cob_description/urdf/cob4_base/base.urdf.xacro (robot description, xacro)
@@ -4,12 +4,12 @@
   <!-- drive_wheel module -->
   <xacro:include filename="$(find cob_description)/urdf/drive_wheel/drive_wheel.urdf.xacro" />
-  <!-- sensors -->
-  <xacro:include filename="$(find cob_description)/urdf/sensors/sick_s300_laser.urdf.xacro"/>
   <!-- properties -->
-  <property name="caster_offset_x" value="0.24844" />  <!--modify here-->
-  <property name="caster_offset_y" value="0.21515" />
-  <property name="caster_offset_z" value="0.08" />
-  <property name="base_mass" value="50" />
+  <xacro:property name="caster_offset_x" value="0.24844" />  <!--modify here-->
+  <xacro:property name="caster_offset_y" value="0.21515" />
+  <xacro:property name="caster_offset_z" value="0.08" />
+  <xacro:property name="base_mass" value="50" />
   <xacro:macro name="base" params="name use_old_joint_names">
+    <xacro:property name="drive_vel" value="19.95" />
+    <xacro:property name="steer_vel" value="117.81" />
     <link name="${name}_footprint"/>
     <joint name="${name}_footprint_joint" type="fixed">
@@ -63,16 +63,13 @@
       </xacro:drive_wheel>
     </xacro:unless>
-    <!-- sensors -->
-    <xacro:sick_s300_laser_v0 name="${name}_laser_front" parent="${name}">
-      <origin xyz="${laser_front_x} ${laser_front_y} ${laser_front_z}" rpy="${laser_front_roll} ${laser_front_pitch} ${laser_front_yaw}" />
-    </xacro:sick_s300_laser_v0>
-    <xacro:sick_s300_laser_v0 name="${name}_laser_left" parent="${name}">
-      <origin xyz="${laser_left_x} ${laser_left_y} ${laser_left_z}" rpy="${laser_left_roll} ${laser_left_pitch} ${laser_left_yaw}" />
-    </xacro:sick_s300_laser_v0>
-    <xacro:sick_s300_laser_v0 name="${name}_laser_right" parent="${name}">
-      <origin xyz="${laser_right_x} ${laser_right_y} ${laser_right_z}" rpy="${laser_right_roll} ${laser_right_pitch} ${laser_right_yaw}" />
-    </xacro:sick_s300_laser_v0>
     <!-- gazebo extensions -->
     <xacro:base_gazebo name="${name}" />
+    <!-- ros_control plugin -->
+    <gazebo>
+      <plugin name="ros_control" filename="libhwi_switch_gazebo_ros_control.so">
+        <robotNamespace>${name}</robotNamespace>
+        <filterJointsParam>joint_names</filterJointsParam>
+      </plugin>
+    </gazebo>
   </xacro:macro>
 </robot>

File: cob_description/urdf/cob4_gripper/gripper.urdf.xacro (robot description, xacro)
@@ -6,5 +6,5 @@
     <!-- joint between base_link and gripper_base_link -->
     <joint name="${name}_base_joint" type="fixed" >
-      <insert_block name="origin" />
+      <xacro:insert_block name="origin" />
       <parent link="${parent}" />
       <child link="${name}_base_link" />
@@ -138,4 +138,11 @@
     <xacro:gripper_gazebo name="${name}" />
     <xacro:gripper_transmission name="${name}" />
+    <!-- ros_control plugin -->
+    <gazebo>
+      <plugin name="ros_control" filename="libhwi_switch_gazebo_ros_control.so">
+        <robotNamespace>${name}</robotNamespace>
+        <filterJointsParam>joint_names</filterJointsParam>
+      </plugin>
+    </gazebo>
   </xacro:macro>
 </robot>

File: cob_description/urdf/cob4_head/head.urdf.xacro (robot description, xacro)
@@ -3,7 +3,7 @@
   <xacro:include filename="$(find cob_description)/urdf/cob4_head/head.gazebo.xacro" />
   <xacro:include filename="$(find cob_description)/urdf/cob4_head/head.transmission.xacro" />
-  <xacro:macro name="head" params="parent name *origin">
+  <xacro:macro name="head" params="parent name *origin dof1:=false dof2:=false dof3:=false">
     <joint name="${name}_base_joint" type="fixed">
-      <insert_block name="origin" />
+      <xacro:insert_block name="origin" />
       <child link="${name}_base_link" />
       <parent link="${parent}"/>
@@ -24,11 +24,20 @@
       </collision>
     </link>
-    <joint name="${name}_1_joint" type="revolute">
-      <origin xyz="0 0 0.0305" rpy="0 0 0"/>
-      <parent link="${name}_base_link"/>
-      <child link="${name}_1_link" />
-      <axis xyz="0 0 1" />
-      <limit effort="100" lower="-6.2831" upper="6.2831" velocity="1.4"/>
-    </joint>
+    <xacro:unless value="${dof1}">
+      <joint name="${name}_1_joint" type="fixed">
+        <origin xyz="0 0 0.0305" rpy="0 0 0"/>
+        <parent link="${name}_base_link"/>
+        <child link="${name}_1_link" />
+      </joint>
+    </xacro:unless>
+    <xacro:if value="${dof1}">
+      <joint name="${name}_1_joint" type="revolute">
+        <origin xyz="0 0 0.0305" rpy="0 0 0"/>
+        <parent link="${name}_base_link"/>
+        <child link="${name}_1_link" />
+        <axis xyz="0 0 1" />
+        <limit effort="100" lower="-6.2831" upper="6.2831" velocity="1.4"/>
+      </joint>
+    </xacro:if>
     <link name="${name}_1_link">
       <xacro:default_inertial/>
@@ -46,11 +55,20 @@
       </collision>
     </link>
-    <joint name="${name}_2_joint" type="revolute">
-      <origin xyz="0 -0.07725 0.00439" rpy="0.349 0 0" />
-      <parent link="${name}_1_link"/>
-      <child link="${name}_2_link" />
-      <axis xyz="0 0 1" />
-      <limit effort="100" lower="-6.2831" upper="6.2831" velocity="1.4"/>
-    </joint>
+    <xacro:unless value="${dof2}">
+      <joint name="${name}_2_joint" type="fixed">
+        <origin xyz="0 -0.07725 0.00439" rpy="0.349 0 0" />
+        <parent link="${name}_1_link"/>
+        <child link="${name}_2_link" />
+      </joint>
+    </xacro:unless>
+    <xacro:if value="${dof2}">
+      <joint name="${name}_2_joint" type="revolute">
+        <origin xyz="0 -0.07725 0.00439" rpy="0.349 0 0" />
+        <parent link="${name}_1_link"/>
+        <child link="${name}_2_link" />
+        <axis xyz="0 0 1" />
+        <limit effort="100" lower="-6.2831" upper="6.2831" velocity="1.4"/>
+      </joint>
+    </xacro:if>
     <link name="${name}_2_link">
       <xacro:default_inertial/>
@@ -68,11 +86,20 @@
       </collision>
     </link>
-    <joint name="${name}_3_joint" type="revolute">
-      <origin xyz="0 0.09849 0.04476" rpy="-0.349 0 0" />
-      <parent link="${name}_2_link"/>
-      <child link="${name}_3_link" />
-      <axis xyz="0 0 1" />
-      <limit effort="100" lower="-6.2831" upper="6.2831" velocity="1.4"/>
-    </joint>
+    <xacro:unless value="${dof3}">
+      <joint name="${name}_3_joint" type="fixed">
+        <origin xyz="0 0.09849 0.04476" rpy="-0.349 0 0" />
+        <parent link="${name}_2_link"/>
+        <child link="${name}_3_link" />
+      </joint>
+    </xacro:unless>
+    <xacro:if value="${dof3}">
+      <joint name="${name}_3_joint" type="revolute">
+        <origin xyz="0 0.09849 0.04476" rpy="-0.349 0 0" />
+        <parent link="${name}_2_link"/>
+        <child link="${name}_3_link" />
+        <axis xyz="0 0 1" />
+        <limit effort="100" lower="-6.2831" upper="6.2831" velocity="1.4"/>
+      </joint>
+    </xacro:if>
     <link name="${name}_3_link">
       <xacro:default_inertial/>
@@ -96,7 +123,16 @@
     </joint>
     <link name="${name}_center_link"/>
-  <!-- extensions -->
-  <xacro:head_gazebo name="${name}" />
-  <xacro:head_transmission name="${name}" />
+    <!-- extensions -->
+    <xacro:head_gazebo name="${name}" />
+    <xacro:head_transmission name="${name}" dof1="${dof1}" dof2="${dof2}" dof3="${dof3}" />
+    <!-- ros_control plugin -->
+    <xacro:if value="${(dof1 == 'true') or (dof2 == 'true') or (dof3 == 'true')}">
+      <gazebo>
+        <plugin name="ros_control" filename="libhwi_switch_gazebo_ros_control.so">
+          <robotNamespace>${name}</robotNamespace>
+          <filterJointsParam>joint_names</filterJointsParam>
+        </plugin>
+      </gazebo>
+    </xacro:if>
   </xacro:macro>
 </robot>

File: cob_description/urdf/cob4_sensorring/sensorring.urdf.xacro (robot description, xacro)
@@ -3,7 +3,7 @@
   <xacro:include filename="$(find cob_description)/urdf/cob4_sensorring/sensorring.gazebo.xacro" />
   <xacro:include filename="$(find cob_description)/urdf/cob4_sensorring/sensorring.transmission.xacro" />
-  <xacro:macro name="sensorring" params="parent name *origin">
+  <xacro:macro name="sensorring" params="parent name *origin active:=false">
     <joint name="${name}_base_joint" type="fixed">
-      <insert_block name="origin" />
+      <xacro:insert_block name="origin" />
       <parent link="${parent}"/>
       <child link="${name}_base_link" />
@@ -24,11 +24,20 @@
       </collision>
     </link>
-    <joint name="${name}_joint" type="revolute">
-      <origin xyz="0 0 0" rpy="0 0 0" />
-      <parent link="${name}_base_link"/>
-      <child link="${name}_link" />
-      <axis xyz="0 0 1" />
-      <limit effort="100" lower="-6.2831" upper="6.2831" velocity="2.62"/>
-    </joint>
+    <xacro:unless value="${active}">
+      <joint name="${name}_joint" type="fixed">
+        <origin xyz="0 0 0" rpy="0 0 0" />
+        <parent link="${name}_base_link"/>
+        <child link="${name}_link" />
+      </joint>
+    </xacro:unless>
+    <xacro:if value="${active}">
+      <joint name="${name}_joint" type="revolute">
+        <origin xyz="0 0 0" rpy="0 0 0" />
+        <parent link="${name}_base_link"/>
+        <child link="${name}_link" />
+        <axis xyz="0 0 1" />
+        <limit effort="100" lower="-6.2831" upper="6.2831" velocity="2.62"/>
+      </joint>
+    </xacro:if>
     <link name="${name}_link">
       <xacro:default_inertial/>
@@ -53,5 +62,14 @@
     <!-- extensions -->
     <xacro:sensorring_gazebo name="${name}" />
-    <xacro:sensorring_transmission name="${name}" />
+    <xacro:sensorring_transmission name="${name}" active="${active}" />
+    <!-- ros_control plugin -->
+    <xacro:if value="${active}">
+      <gazebo>
+        <plugin name="ros_control" filename="libhwi_switch_gazebo_ros_control.so">
+          <robotNamespace>${name}</robotNamespace>
+          <filterJointsParam>joint_names</filterJointsParam>
+        </plugin>
+      </gazebo>
+    </xacro:if>
   </xacro:macro>
 </robot>

File: cob_description/urdf/cob4_torso/torso.urdf.xacro (robot description, xacro)
@@ -3,9 +3,7 @@
   <xacro:include filename="$(find cob_description)/urdf/cob4_torso/torso.gazebo.xacro" />
   <xacro:include filename="$(find cob_description)/urdf/cob4_torso/torso.transmission.xacro" />
-  <xacro:include filename="$(find cob_description)/urdf/sensors/softkinetic.urdf.xacro" />
-  <xacro:include filename="$(find cob_description)/urdf/sensors/kinect.urdf.xacro" />
-  <xacro:macro name="torso" params="parent name *origin">
+  <xacro:macro name="torso" params="parent name *origin dof1:=false dof2:=false dof3:=false">
     <joint name="${name}_base_joint" type="fixed">
-      <insert_block name="origin" />
+      <xacro:insert_block name="origin" />
       <parent link="${parent}"/>
       <child link="${name}_base_link" />
@@ -31,11 +29,20 @@
       </collision>
     </link>
-    <joint name="${name}_1_joint" type="revolute">
-      <origin xyz="0 0 0.04642" rpy="0 0 0"/>
-      <parent link="${name}_base_link"/>
-      <child link="${name}_1_link" />
-      <axis xyz="0 0 1" />
-      <limit effort="100" lower="-6.2831" upper="6.2831" velocity="1.4"/>
-    </joint>
+    <xacro:unless value="${dof1}">
+      <joint name="${name}_1_joint" type="fixed">
+        <origin xyz="0 0 0.04642" rpy="0 0 0"/>
+        <parent link="${name}_base_link"/>
+        <child link="${name}_1_link" />
+      </joint>
+    </xacro:unless>
+    <xacro:if value="${dof1}">
+      <joint name="${name}_1_joint" type="revolute">
+        <origin xyz="0 0 0.04642" rpy="0 0 0"/>
+        <parent link="${name}_base_link"/>
+        <child link="${name}_1_link" />
+        <axis xyz="0 0 1" />
+        <limit effort="100" lower="-6.2831" upper="6.2831" velocity="1.4"/>
+      </joint>
+    </xacro:if>
     <link name="${name}_1_link">
       <xacro:default_inertial/>
@@ -58,11 +65,20 @@
       </collision>
     </link>
-    <joint name="${name}_2_joint" type="revolute">
-      <origin xyz="0 0.14734 0.07547" rpy="0.5236 0 0" />
-      <parent link="${name}_1_link"/>
-      <child link="${name}_2_link" />
-      <axis xyz="0 0 1" />
-      <limit effort="100" lower="-6.2831" upper="6.2831" velocity="1.4"/>
-    </joint>
+    <xacro:unless value="${dof2}">
+      <joint name="${name}_2_joint" type="fixed">
+        <origin xyz="0 0.14734 0.07547" rpy="0.5236 0 0" />
+        <parent link="${name}_1_link"/>
+        <child link="${name}_2_link" />
+      </joint>
+    </xacro:unless>
+    <xacro:if value="${dof2}">
+      <joint name="${name}_2_joint" type="revolute">
+        <origin xyz="0 0.14734 0.07547" rpy="0.5236 0 0" />
+        <parent link="${name}_1_link"/>
+        <child link="${name}_2_link" />
+        <axis xyz="0 0 1" />
+        <limit effort="100" lower="-6.2831" upper="6.2831" velocity="1.4"/>
+      </joint>
+    </xacro:if>
     <link name="${name}_2_link">
       <xacro:default_inertial/>
@@ -85,11 +101,20 @@
       </collision>
     </link>
-    <joint name="${name}_3_joint" type="revolute">
-      <origin xyz="0 -0.09228 0.13477" rpy="-0.5236 0 0" />
-      <parent link="${name}_2_link"/>
-      <child link="${name}_3_link" />
-      <axis xyz="0 0 1" />
-      <limit effort="100" lower="-6.2831" upper="6.2831" velocity="1.4"/>
-    </joint>
+    <xacro:unless value="${dof3}">
+      <joint name="${name}_3_joint" type="fixed">
+        <origin xyz="0 -0.09228 0.13477" rpy="-0.5236 0 0" />
+        <parent link="${name}_2_link"/>
+        <child link="${name}_3_link" />
+      </joint>
+    </xacro:unless>
+    <xacro:if value="${dof3}">
+      <joint name="${name}_3_joint" type="revolute">
+        <origin xyz="0 -0.09228 0.13477" rpy="-0.5236 0 0" />
+        <parent link="${name}_2_link"/>
+        <child link="${name}_3_link" />
+        <axis xyz="0 0 1" />
+        <limit effort="100" lower="-6.2831" upper="6.2831" velocity="1.4"/>
+      </joint>
+    </xacro:if>
     <link name="${name}_3_link">
       <xacro:default_inertial/>
@@ -132,19 +157,16 @@
       </collision>
     </link>
-    <!-- left camera -->
-    <xacro:cob_kinect_v0 name="${name}_cam3d_left" ros_topic="torso_cam3d_left" parent="${name}_3_link">
-      <origin xyz="${torso_cam3d_left_x} ${torso_cam3d_left_y} ${torso_cam3d_left_z}" rpy="${torso_cam3d_left_roll} ${torso_cam3d_left_pitch} ${torso_cam3d_left_yaw}" />
-    </xacro:cob_kinect_v0>
-    <!-- right camera -->
-    <xacro:cob_kinect_v0 name="${name}_cam3d_right" ros_topic="torso_cam3d_right" parent="${name}_3_link">
-      <origin xyz="${torso_cam3d_right_x} ${torso_cam3d_right_y} ${torso_cam3d_right_z}" rpy="${torso_cam3d_right_roll} ${torso_cam3d_right_pitch} ${torso_cam3d_right_yaw}" />
-    </xacro:cob_kinect_v0>
-    <!-- down camera -->
-    <xacro:softkinetic name="${name}_cam3d_down" ros_topic="torso_cam3d_down" parent="${name}_3_link">
-      <origin xyz="${torso_cam3d_down_x} ${torso_cam3d_down_y} ${torso_cam3d_down_z}" rpy="${torso_cam3d_down_roll} ${torso_cam3d_down_pitch} ${torso_cam3d_down_yaw}" />
-    </xacro:softkinetic>
     <!-- extensions -->
-    <xacro:torso_gazebo name="torso" />
-    <xacro:torso_transmission name="torso" />
+    <xacro:torso_gazebo name="${name}" />
+    <xacro:torso_transmission name="${name}" dof1="${dof1}" dof2="${dof2}" dof3="${dof3}" />
+    <!-- ros_control plugin -->
+    <xacro:if value="${(dof1 == 'true') or (dof2 == 'true') or (dof3 == 'true')}">
+      <gazebo>
+        <plugin name="ros_control" filename="libhwi_switch_gazebo_ros_control.so">
+          <robotNamespace>${name}</robotNamespace>
+          <filterJointsParam>joint_names</filterJointsParam>
+        </plugin>
+      </gazebo>
+    </xacro:if>
   </xacro:macro>
 </robot>

File: cob_description/urdf/drive_wheel/drive_wheel.urdf.xacro (robot description, xacro)
@@ -3,8 +3,8 @@
   <xacro:include filename="$(find cob_description)/urdf/drive_wheel/drive_wheel.gazebo.xacro" />
   <xacro:include filename="$(find cob_description)/urdf/drive_wheel/drive_wheel.transmission.xacro" />
-  <property name="caster_wheel_offset_y" value="0.0" />
-  <property name="caster_mass" value="5.9" />
-  <property name="wheel_mass" value="0.44036" />
-  <xacro:macro name="cob_wheel" params="parent suffix reflect">
+  <xacro:property name="caster_wheel_offset_y" value="0.0" />
+  <xacro:property name="caster_mass" value="5.9" />
+  <xacro:property name="wheel_mass" value="0.44036" />
+  <xacro:macro name="cob_wheel" params="parent suffix reflect drive_vel:=^">
     <joint name="${parent}_${suffix}_wheel_joint" type="continuous">
       <origin xyz="0 ${reflect*caster_wheel_offset_y} 0" rpy="0 0 0" />
@@ -12,6 +12,6 @@
       <child link="${parent}_${suffix}_wheel_link"/>
       <axis xyz="0 1 0" />
-      <limit effort="100" velocity="100"/> <!-- alpha tested effort and velocity limits -->
       <safety_controller  k_velocity="10" />
+      <limit effort="100" velocity="${drive_vel}"/>
       <dynamics damping="0.0" friction="0.0" />
     </joint>
@@ -39,12 +39,12 @@
   </xacro:macro>
   <!-- Macro for Caster hub only -->
-  <xacro:macro name="cob_caster_hub" params="*origin parent suffix" >
+  <xacro:macro name="cob_caster_hub" params="*origin parent suffix steer_vel:=^" >
     <joint name="${suffix}_rotation_joint" type="continuous">
-      <insert_block name="origin" />
+      <xacro:insert_block name="origin" />
       <parent link="${parent}"/>
       <child link="${suffix}_rotation_link" />
       <axis xyz="0 0 1" />
-      <limit effort="100" velocity="100"/> <!-- alpha tested velocity and effort limits -->
       <safety_controller  k_velocity="10" />
+      <limit effort="100" velocity="${steer_vel}"/>
       <dynamics damping="0.0" friction="0.0" />
     </joint>
@@ -71,7 +71,7 @@
     <xacro:cob_caster_transmission suffix="${suffix}" />
   </xacro:macro>
-  <xacro:macro name="drive_wheel" params="*origin parent suffix">
+  <xacro:macro name="drive_wheel" params="*origin parent suffix drive_vel:=^|100 steer_vel:=^|100">
     <xacro:cob_caster_hub parent="${parent}" suffix="${suffix}_caster" >
-      <insert_block name="origin" />
+      <xacro:insert_block name="origin" />
     </xacro:cob_caster_hub>
     <xacro:cob_wheel parent="${suffix}_caster" suffix="r" reflect="-1" />

File: cob_description/urdf/sensors/kinect.gazebo.xacro (robot description, xacro)
@@ -1,15 +1,16 @@
 <?xml version="1.0"?>
 <root xmlns:xacro="http://www.ros.org/wiki/xacro">
-  <xacro:macro name="cob_kinect_gazebo_v0" params="name ros_topic">
+  <xacro:macro name="cob_kinect_gazebo_v0" params="name ros_topic
+                                                   update_rate:=20 data_skip:=0 height:=480 width:=640">
     <gazebo reference="${name}_frame">
       <sensor type="depth" name="${name}_frame_sensor">
         <always_on>true</always_on>
-        <update_rate>20.0</update_rate>
+        <update_rate>${update_rate/(data_skip+1)}</update_rate>
         <camera>
           <horizontal_fov>${62.0*M_PI/180.0}</horizontal_fov>
           <image>
             <format>R8G8B8</format>
-            <width>640</width>
-            <height>480</height>
+            <width>${height}</width>
+            <height>${width}</height>
           </image>
           <clip>
@@ -24,5 +25,5 @@
         </camera>
         <plugin name="${name}_controller" filename="libgazebo_ros_openni_kinect.so">
-          <updateRate>20.0</updateRate>
+          <updateRate>${update_rate/(data_skip+1)}</updateRate>
           <cameraName>${ros_topic}</cameraName>
           <frameName>${name}_link</frameName>

File: cob_description/urdf/sensors/kinect.urdf.xacro (robot description, xacro)
@@ -2,7 +2,7 @@
 <root xmlns:xacro="http://www.ros.org/wiki/xacro">
   <xacro:include filename="$(find cob_description)/urdf/sensors/kinect.gazebo.xacro" />
-  <xacro:macro name="cob_kinect_v0" params="name parent *origin ros_topic">
+  <xacro:macro name="cob_kinect_v0" params="name parent *origin ros_topic update_rate:=20 data_skip:=0 height:=480 width:=640">
     <joint name="${name}_joint" type="fixed">
-      <insert_block name="origin" />
+      <xacro:insert_block name="origin" />
       <parent link="${parent}"/>
       <child link="${name}_link"/>
@@ -33,5 +33,9 @@
     <link name="${name}_frame"/>
     <!-- extensions -->
-    <xacro:cob_kinect_gazebo_v0 name="${name}" ros_topic="${ros_topic}" />
+    <xacro:cob_kinect_gazebo_v0 name="${name}" ros_topic="${ros_topic}"
+    									       update_rate="${update_rate}"
+    									       data_skip="${data_skip}"
+									           height="${height}"
+									           width="${width}"/>
   </xacro:macro>
 </root>

File: cob_description/urdf/sensors/realsense.gazebo.xacro (robot description, xacro)
@@ -1,15 +1,18 @@
 <?xml version="1.0"?>
 <robot xmlns:xacro="http://www.ros.org/wiki/xacro">
-  <xacro:macro name="realsense_gazebo" params="name ros_topic">
+  <!-- use default values of realsense_camera/r200_nodelet_rgbd -->
+  <xacro:macro name="realsense_gazebo" params="name ros_topic
+                                               depth_fps:=30.0 depth_height:=360 depth_width:=480
+                                               color_fps:=30.0 color_height:=480 color_width:=640" >
     <gazebo reference="${name}_link">
       <sensor type="depth" name="${name}_depth_frame">
         <always_on>true</always_on>
-        <update_rate>25.0</update_rate>
+        <update_rate>${color_fps}</update_rate>
         <camera>
           <horizontal_fov>${74.0*M_PI/180.0}</horizontal_fov>
           <image>
             <format>R8G8B8</format>
-            <width>320</width>
-            <height>240</height>
+            <width>${color_width}</width>
+            <height>${color_height}</height>
           </image>
           <clip>
@@ -24,5 +27,5 @@
         </camera>
         <plugin name="${name}_frame_controller" filename="libgazebo_ros_openni_kinect.so">
-          <updateRate>25.0</updateRate>
+          <updateRate>${color_fps}</updateRate>
           <cameraName>${ros_topic}</cameraName>
           <frameName>${name}_rgb_optical_frame</frameName>

File: cob_description/urdf/sensors/sick_s300_laser.gazebo.xacro (robot description, xacro)
@@ -25,5 +25,5 @@
             <type>gaussian</type>
             <mean>0.0</mean>
-            <stddev>0.005</stddev>
+            <stddev>0.02</stddev>
           </noise>
         </ray>
