Commit message: Imported upstream version '0.6.7' of 'upstream'

File: cob_description/urdf/sensors/usb_cam.urdf.xacro (robot description, xacro)
@@ -1,6 +1,6 @@
 <?xml version="1.0"?>
 <robot xmlns:xacro="http://www.ros.org/wiki/xacro">
-  <xacro:include filename="$(find cob_description)/urdf/sensors/realsense.gazebo.xacro" />
-  <xacro:macro name="realsense" params="name parent ros_topic *origin">
+  <xacro:include filename="$(find cob_description)/urdf/sensors/usb_cam.gazebo.xacro" />
+  <xacro:macro name="usb_cam" params="name parent *origin ros_topic update_rate height width">
     <joint name="${name}_joint" type="fixed">
       <xacro:insert_block name="origin" />
@@ -10,5 +10,5 @@
     <link name="${name}_link">
       <inertial>
-        <mass value="0.564" />
+        <mass value="0.1" />
         <origin xyz="0 0 0" />
         <inertia ixx="0.003881243" ixy="0.0" ixz="0.0" iyy="0.000498940" iyz="0.0" izz="0.003879257" />
@@ -27,6 +27,15 @@
       </collision>
     </link>
+    <joint name="${name}_frame_joint" type="fixed">
+      <origin xyz="0 0 0" rpy="${M_PI/2} -${M_PI/2} 0" />
+      <parent link="${name}_link"/>
+      <child link="${name}_frame"/>
+    </joint>
+    <link name="${name}_frame"/>
     <!-- extensions -->
-    <xacro:realsense_gazebo name="${name}" ros_topic="${ros_topic}" />
+    <xacro:usb_cam_gazebo name="${name}" ros_topic="${ros_topic}"
+									     update_rate="${update_rate}"
+									     height="${height}"
+									     width="${width}"/>
   </xacro:macro>
 </robot>

File: cob_description/urdf/ur_arm/ur10_arm.urdf.xacro (robot description, xacro)
@@ -3,9 +3,8 @@
   <xacro:include filename="$(find cob_description)/urdf/common.xacro" />
   <xacro:include filename="$(find ur_description)/urdf/ur10.urdf.xacro" />
-  <!--property name="wrist_3_length" value="0.0857" /-->
   <xacro:macro name="ur10" params="parent name *origin">
     <!-- mount the arm to the robot -->
     <joint name="${name}_base_joint" type="fixed" >
-      <insert_block name="origin" />
+      <xacro:insert_block name="origin" />
       <parent link="${parent}" />
       <child link="${name}_base_link" />
@@ -13,4 +12,11 @@
     <!-- include universal_robot arm -->
     <xacro:ur10_robot prefix="${name}_" joint_limited="true"/>
+    <!-- ros_control plugin -->
+    <gazebo>
+      <plugin name="ros_control" filename="libhwi_switch_gazebo_ros_control.so">
+        <robotNamespace>${name}</robotNamespace>
+        <filterJointsParam>joint_names</filterJointsParam>
+      </plugin>
+    </gazebo>
   </xacro:macro>
 </robot>

File: cob_description/urdf/ur_arm/ur5_arm.urdf.xacro (robot description, xacro)
@@ -3,9 +3,8 @@
   <xacro:include filename="$(find cob_description)/urdf/common.xacro" />
   <xacro:include filename="$(find ur_description)/urdf/ur5.urdf.xacro" />
-  <!--property name="wrist_3_length" value="0.0823" /-->
   <xacro:macro name="ur5" params="parent name *origin">
     <!-- mount the arm to the robot -->
     <joint name="${name}_base_joint" type="fixed" >
-      <insert_block name="origin" />
+      <xacro:insert_block name="origin" />
       <parent link="${parent}" />
       <child link="${name}_base_link" />
@@ -13,4 +12,11 @@
     <!-- include universal_robot arm -->
     <xacro:ur5_robot prefix="${name}_" joint_limited="true"/>
+    <!-- ros_control plugin -->
+    <gazebo>
+      <plugin name="ros_control" filename="libhwi_switch_gazebo_ros_control.so">
+        <robotNamespace>${name}</robotNamespace>
+        <filterJointsParam>joint_names</filterJointsParam>
+      </plugin>
+    </gazebo>
   </xacro:macro>
 </robot>

File: raw_description/urdf/base_long/base.urdf.xacro (robot description, xacro)
@@ -5,28 +5,25 @@
   <!-- drive_wheel module -->
   <xacro:include filename="$(find cob_description)/urdf/drive_wheel/drive_wheel.urdf.xacro" />
-  <!-- sensors -->
-  <xacro:include filename="$(find cob_description)/urdf/sensors/sick_s300_laser.urdf.xacro"/>
-  <xacro:include filename="$(find cob_description)/urdf/sensors/kinect.urdf.xacro"/>
   <!-- properties -->
-  <property name="caster_offset_x" value="0.368" />  <!--modify here-->
-  <property name="caster_offset_y_bl" value="0.134" />
-  <property name="caster_offset_y_br" value="-0.184" />
-  <property name="caster_offset_y_fl" value="0.184" />
-  <property name="caster_offset_y_fr" value="-0.134" />
-  <property name="caster_offset_z" value="0.09" />
-  <property name="battery_offset_x_f" value="0.141" />
-  <property name="battery_offset_x_r" value="0.139" />
-  <property name="battery_offset_y_f" value="-0.008" />
-  <property name="battery_offset_y_r" value="0.007" />
-  <property name="battery_offset_z" value="0.065" />
-  <property name="base_mass" value="83.1" />
-  <property name="battery_mass" value="25.0" />
-  <property name="battery_size_x" value="0.5" />
-  <property name="battery_size_y" value="0.148" />
-  <property name="battery_size_z" value="0.26" />
+  <xacro:property name="caster_offset_x" value="0.368" />  <!--modify here-->
+  <xacro:property name="caster_offset_y_bl" value="0.134" />
+  <xacro:property name="caster_offset_y_br" value="-0.184" />
+  <xacro:property name="caster_offset_y_fl" value="0.184" />
+  <xacro:property name="caster_offset_y_fr" value="-0.134" />
+  <xacro:property name="caster_offset_z" value="0.08" />
+  <xacro:property name="battery_offset_x_f" value="0.141" />
+  <xacro:property name="battery_offset_x_r" value="0.139" />
+  <xacro:property name="battery_offset_y_f" value="-0.008" />
+  <xacro:property name="battery_offset_y_r" value="0.007" />
+  <xacro:property name="battery_offset_z" value="0.065" />
+  <xacro:property name="base_mass" value="83.1" />
+  <xacro:property name="battery_mass" value="50.0" />
+  <xacro:property name="battery_size_x" value="0.5" />
+  <xacro:property name="battery_size_y" value="0.148" />
+  <xacro:property name="battery_size_z" value="0.26" />
   <!-- battery macros-->
   <xacro:macro name="cob_batteries" params="name parent *origin ">
     <joint name="${name}_battery_joint" type="fixed">
-      <insert_block name="origin" />
+      <xacro:insert_block name="origin" />
       <parent link="${parent}"/>
       <child link="${name}_battery" />
@@ -34,5 +31,5 @@
     <link name="${name}_battery">
       <xacro:box_inertial x="${battery_size_x}" y="${battery_size_y}" z="${battery_size_z}" mass="${battery_mass}">
-        <origin xyz="0 0 0" rpy="0 0 0" />
+        <origin xyz="0 0 0" rpy="0 0 0"/>
       </xacro:box_inertial>
       <visual>
@@ -62,10 +59,7 @@
     </joint>
     <link name="${name}_link">
-      <inertial>
-        <origin xyz="0 0 0" />
-        <mass value="${base_mass}" />
-        <inertia ixx="9.64" ixy="-0.02" ixz="0.44"
-                 iyy="11.33" iyz="-0.007" izz="3.07" />
-      </inertial>
+      <xacro:box_inertial x="1.04" y="0.58" z="0.12" mass="${base_mass}">
+        <origin xyz="0 0 0" rpy="0 0 0"/>
+      </xacro:box_inertial>
       <visual>
         <origin xyz="0 0 0.209" rpy="0 0 0" />
@@ -95,16 +89,4 @@
       <origin xyz="${-caster_offset_x} ${caster_offset_y_br} ${caster_offset_z}" rpy="0 0 0" />
     </xacro:drive_wheel>
-    <!-- base laser front -->
-    <xacro:sick_s300_laser_v0 name="${name}_laser_front" parent="${name}">
-      <origin xyz="${laser_front_x} ${laser_front_y} ${laser_front_z}" rpy="${laser_front_roll} ${laser_front_pitch} ${laser_front_yaw}" />
-    </xacro:sick_s300_laser_v0>
-    <!-- base laser rear -->
-    <xacro:sick_s300_laser_v0 name="${name}_laser_rear" parent="${name}">
-      <origin xyz="${laser_rear_x} ${laser_rear_y} ${laser_rear_z}" rpy="${laser_rear_roll} ${laser_rear_pitch} ${laser_rear_yaw}" />
-    </xacro:sick_s300_laser_v0>
-    <!-- cam3d -->
-    <!--xacro:cob_kinect_v0 name="${name}_cam3d" ros_topic="cam3d" parent="${name}_link">
-      <origin xyz="0.51 0.12 0.27" rpy="-${M_PI/2} 0 -${M_PI/2}" />
-    </xacro:cob_kinect_v0-->
     <!-- battery front-->
     <xacro:cob_batteries name="${name}_battery_front" parent="${name}_link">
@@ -117,4 +99,11 @@
     <!-- gazebo extensions -->
     <xacro:base_gazebo name="${name}" />
+    <!-- ros_control plugin -->
+    <gazebo>
+      <plugin name="ros_control" filename="libhwi_switch_gazebo_ros_control.so">
+        <robotNamespace>${name}</robotNamespace>
+        <filterJointsParam>joint_names</filterJointsParam>
+      </plugin>
+    </gazebo>
   </xacro:macro>
 </robot>

File: raw_description/urdf/base_short/base.urdf.xacro (robot description, xacro)
@@ -5,26 +5,23 @@
   <!-- drive_wheel module -->
   <xacro:include filename="$(find cob_description)/urdf/drive_wheel/drive_wheel.urdf.xacro" />
-  <!-- sensors -->
-  <xacro:include filename="$(find cob_description)/urdf/sensors/sick_s300_laser.urdf.xacro"/>
-  <xacro:include filename="$(find cob_description)/urdf/sensors/kinect.urdf.xacro"/>
   <!-- properties -->
-  <property name="caster_offset_x" value="0.228" />  <!--modify here-->
-  <property name="caster_offset_y_bl" value="0.134" />
-  <property name="caster_offset_y_br" value="-0.184" />
-  <property name="caster_offset_y_fl" value="0.184" />
-  <property name="caster_offset_y_fr" value="-0.134" />
-  <property name="caster_offset_z" value="0.09" />
-  <property name="battery_offset_x" value="0.0" />
-  <property name="battery_offset_y" value="-0.008" />
-  <property name="battery_offset_z" value="0.065" />
-  <property name="base_mass" value="43.1" />
-  <property name="battery_mass" value="40" />
-  <property name="battery_size_x" value="0.5" />
-  <property name="battery_size_y" value="0.148" />
-  <property name="battery_size_z" value="0.26" />
+  <xacro:property name="caster_offset_x" value="0.228" />  <!--modify here-->
+  <xacro:property name="caster_offset_y_bl" value="0.134" />
+  <xacro:property name="caster_offset_y_br" value="-0.184" />
+  <xacro:property name="caster_offset_y_fl" value="0.184" />
+  <xacro:property name="caster_offset_y_fr" value="-0.134" />
+  <xacro:property name="caster_offset_z" value="0.08" />
+  <xacro:property name="battery_offset_x" value="0.0" />
+  <xacro:property name="battery_offset_y" value="-0.008" />
+  <xacro:property name="battery_offset_z" value="0.065" />
+  <xacro:property name="base_mass" value="43.1" />
+  <xacro:property name="battery_mass" value="40" />
+  <xacro:property name="battery_size_x" value="0.5" />
+  <xacro:property name="battery_size_y" value="0.148" />
+  <xacro:property name="battery_size_z" value="0.26" />
   <!-- battery macros-->
   <xacro:macro name="cob_batteries" params="name parent *origin ">
     <joint name="${name}_battery_joint" type="fixed">
-      <insert_block name="origin" />
+      <xacro:insert_block name="origin" />
       <parent link="${parent}"/>
       <child link="${name}_battery" />
@@ -96,16 +93,4 @@
       <origin xyz="${-caster_offset_x} ${caster_offset_y_br} ${caster_offset_z}" rpy="0 0 0" />
     </xacro:drive_wheel>
-    <!-- base laser front -->
-    <xacro:sick_s300_laser_v0 name="${name}_laser_front" parent="${name}">
-      <origin xyz="${laser_front_x} ${laser_front_y} ${laser_front_z}" rpy="${laser_front_roll} ${laser_front_pitch} ${laser_front_yaw}" />
-    </xacro:sick_s300_laser_v0>
-    <!-- base laser rear -->
-    <xacro:sick_s300_laser_v0 name="${name}_laser_rear" parent="${name}">
-      <origin xyz="${laser_rear_x} ${laser_rear_y} ${laser_rear_z}" rpy="${laser_rear_roll} ${laser_rear_pitch} ${laser_rear_yaw}" />
-    </xacro:sick_s300_laser_v0>
-    <!-- cam3d -->
-    <!--xacro:cob_kinect_v0 name="${name}_cam3d" ros_topic="cam3d" parent="${name}_link">
-      <origin xyz="0.51 0.12 0.27" rpy="-${M_PI/2} 0 -${M_PI/2}" />
-    </xacro:cob_kinect_v0-->
     <!-- battery-->
     <xacro:cob_batteries name="${name}_battery" parent="${name}_link">
@@ -114,4 +99,11 @@
     <!-- gazebo extensions -->
     <xacro:base_gazebo name="${name}" />
+    <!-- ros_control plugin -->
+    <gazebo>
+      <plugin name="ros_control" filename="libhwi_switch_gazebo_ros_control.so">
+        <robotNamespace>${name}</robotNamespace>
+        <filterJointsParam>joint_names</filterJointsParam>
+      </plugin>
+    </gazebo>
   </xacro:macro>
 </robot>

File: raw_description/urdf/torso/torso.urdf.xacro (robot description, xacro)
@@ -6,5 +6,5 @@
     <!-- joint between base_link and torso_tilt_link -->
     <joint name="${name}_0_joint" type="fixed" >
-      <insert_block name="origin" />
+      <xacro:insert_block name="origin" />
       <parent link="${parent}" />
       <child link="${name}_0_link" />
@@ -64,5 +64,5 @@
          <parent link="${name}_1_link"/>
       <child link="torso_2_link"/>
-      <axis xyz="0 1.0 0" />
+      <axis xyz="-1.0 0 0" />
       <dynamics damping="0.1" />
       <limit effort="100" lower="-3.2" upper="1.57" velocity="1.4"/>
@@ -91,4 +91,11 @@
     <xacro:raw_torso_gazebo name="${name}" />
     <xacro:raw_torso_transmission name="${name}" />
+    <!-- ros_control plugin -->
+    <gazebo>
+      <plugin name="ros_control" filename="libhwi_switch_gazebo_ros_control.so">
+        <robotNamespace>${name}</robotNamespace>
+        <filterJointsParam>joint_names</filterJointsParam>
+      </plugin>
+    </gazebo>
   </xacro:macro>
 </robot>

File: raw_description/urdf/vacuum_gripper/gripper.gazebo.xacro (robot description, xacro)
@@ -1,9 +1,8 @@
 <?xml version="1.0"?>
 <robot xmlns:xacro="http://www.ros.org/wiki/xacro">
-  <xacro:macro name="head_gazebo" params="name">
-    <gazebo reference="${name}_axis_link">
+  <xacro:macro name="vacuum_gripper_gazebo" params="name">
+    <gazebo reference="${name}_ee_link">
       <gravity>true</gravity>
       <self_collide>false</self_collide>
-      <material>IPA/LightGrey</material>
     </gazebo>
   </xacro:macro>

Commit message: Imported upstream version '0.6.9' of 'upstream'

File: cob_description/urdf/cob4_base/base.urdf.xacro (robot description, xacro)
@@ -7,7 +7,7 @@
   <xacro:property name="caster_offset_x" value="0.24844" />  <!--modify here-->
   <xacro:property name="caster_offset_y" value="0.21515" />
-  <xacro:property name="caster_offset_z" value="0.08" />
+  <xacro:property name="caster_offset_z" value="0.0782" />
   <xacro:property name="base_mass" value="100" />
-  <xacro:macro name="base" params="name tricycle_mode:=false">
+  <xacro:macro name="base" params="name tricycle_mode:=false drive_dir_angle:=0">
     <xacro:property name="drive_vel" value="19.95" />
     <xacro:property name="steer_vel" value="117.81" />
@@ -18,5 +18,11 @@
       <child link="${name}_link" />
     </joint>
-    <link name="${name}_link">
+    <link name="${name}_link"/>
+    <joint name="${name}_chassis_joint" type="fixed">
+      <origin xyz="0 0 0" rpy="0 0 ${drive_dir_angle}" />
+      <parent link="${name}_link"/>
+      <child link="${name}_chassis_link" />
+    </joint>
+    <link name="${name}_chassis_link">
       <inertial>
         <origin xyz="0 0 0" />
@@ -40,24 +46,30 @@
       </collision>
     </link>
+    <joint name="${name}_charger_joint" type="fixed">
+      <origin xyz="0.2992 0.0 0.09089" rpy="0 0 0" />
+      <parent link="${name}_chassis_link"/>
+      <child link="${name}_charger_link" />
+    </joint>
+    <link name="${name}_charger_link"/>
     <!-- arrangement of the three drive_wheel modules -->
     <xacro:if value="${tricycle_mode}">
-      <xacro:drive_wheel parent="${name}_link" suffix="fl" passive="true" >
+      <xacro:drive_wheel parent="${name}_chassis_link" suffix="fl" passive="true" >
         <origin xyz="${caster_offset_x/2} ${caster_offset_y} ${caster_offset_z}" rpy="0 0 0" />
       </xacro:drive_wheel>
-      <xacro:drive_wheel parent="${name}_link" suffix="b" >
+      <xacro:drive_wheel parent="${name}_chassis_link" suffix="b" >
         <origin xyz="${-caster_offset_x} 0.0 ${caster_offset_z}" rpy="0 0 0" />
       </xacro:drive_wheel>
-      <xacro:drive_wheel parent="${name}_link" suffix="fr" passive="true">
+      <xacro:drive_wheel parent="${name}_chassis_link" suffix="fr" passive="true">
         <origin xyz="${caster_offset_x/2} ${-caster_offset_y} ${caster_offset_z}" rpy="0 0 0" />
       </xacro:drive_wheel>
     </xacro:if>
     <xacro:unless value="${tricycle_mode}">
-      <xacro:drive_wheel parent="${name}_link" suffix="fl" >
+      <xacro:drive_wheel parent="${name}_chassis_link" suffix="fl" >
         <origin xyz="${caster_offset_x/2} ${caster_offset_y} ${caster_offset_z}" rpy="0 0 0" />
       </xacro:drive_wheel>
-      <xacro:drive_wheel parent="${name}_link" suffix="b" >
+      <xacro:drive_wheel parent="${name}_chassis_link" suffix="b" >
         <origin xyz="${-caster_offset_x} 0.0 ${caster_offset_z}" rpy="0 0 0" />
       </xacro:drive_wheel>
-      <xacro:drive_wheel parent="${name}_link" suffix="fr" >
+      <xacro:drive_wheel parent="${name}_chassis_link" suffix="fr" >
         <origin xyz="${caster_offset_x/2} ${-caster_offset_y} ${caster_offset_z}" rpy="0 0 0" />
       </xacro:drive_wheel>

File: raw_description/urdf/torso/torso_v2.urdf.xacro (robot description, xacro)
@@ -10,21 +10,15 @@
     </joint>
     <link name="${name}_0_link">
-      <inertial>
-        <origin xyz="0 0 0.254" rpy="0 0 0"/>
-        <mass value="0.57307"/>
-        <inertia ixx="1.415" ixy="0" ixz="0" iyy="0.819" iyz="0" izz="0.819" />
-      </inertial>
+      <xacro:cylinder_inertial radius="0.04" length="0.508" mass="1.0">
+        <origin xyz="0 0 0.254" rpy="0 0 0" />
+      </xacro:cylinder_inertial>
       <visual>
         <origin xyz="0 0 0.254" rpy="0 0 0" />
-        <geometry>
-          <cylinder length="0.508" radius="0.04"/>
-        </geometry>
+        <xacro:cylinder_geometry radius="0.04" length="0.508" />
         <material name="IPA/LightGrey" />
       </visual>
       <collision>
         <origin xyz="0 0 0.254" rpy="0 0 0" />
-        <geometry>
-          <cylinder length="0.508" radius="0.04"/>
-        </geometry>
+        <xacro:cylinder_geometry radius="0.04" length="0.508" />
       </collision>
     </link>

Commit message: Imported upstream version '0.6.10' of 'upstream'

File: cob_description/urdf/cob4_base/base.urdf.xacro (robot description, xacro)
@@ -9,7 +9,24 @@
   <xacro:property name="caster_offset_z" value="0.0782" />
   <xacro:property name="base_mass" value="100" />
-  <xacro:macro name="base" params="name tricycle_mode:=false drive_dir_angle:=0">
+  <xacro:macro name="base" params="name tricycle_mode:=false forward:=true">
     <xacro:property name="drive_vel" value="19.95" />
     <xacro:property name="steer_vel" value="117.81" />
+    <xacro:if value="${tricycle_mode}">
+      <link name="${name}_pivot_link"/>
+      <xacro:if value="${forward}">
+        <joint name="${name}_pivot_joint" type="fixed">
+          <origin xyz="${-caster_offset_x/2} 0.0 0.0" rpy="0 0 0" />
+          <parent link="${name}_pivot_link"/>
+          <child link="${name}_footprint" />
+        </joint>
+      </xacro:if>
+      <xacro:unless value="${forward}">
+        <joint name="${name}_pivot_joint" type="fixed">
+          <origin xyz="${caster_offset_x/2} 0.0 0.0" rpy="0 0 0" />
+          <parent link="${name}_pivot_link"/>
+          <child link="${name}_footprint" />
+        </joint>
+      </xacro:unless>
+    </xacro:if>
     <link name="${name}_footprint"/>
     <joint name="${name}_footprint_joint" type="fixed">
@@ -19,9 +36,18 @@
     </joint>
     <link name="${name}_link"/>
-    <joint name="${name}_chassis_joint" type="fixed">
-      <origin xyz="0 0 0" rpy="0 0 ${drive_dir_angle}" />
-      <parent link="${name}_link"/>
-      <child link="${name}_chassis_link" />
-    </joint>
+    <xacro:if value="${forward}">
+      <joint name="${name}_chassis_joint" type="fixed">
+        <origin xyz="0 0 0" rpy="0 0 0" />
+        <parent link="${name}_link"/>
+        <child link="${name}_chassis_link" />
+      </joint>
+    </xacro:if>
+    <xacro:unless value="${forward}">
+      <joint name="${name}_chassis_joint" type="fixed">
+        <origin xyz="0 0 0" rpy="0 0 ${M_PI}" />
+        <parent link="${name}_link"/>
+        <child link="${name}_chassis_link" />
+      </joint>
+    </xacro:unless>
     <link name="${name}_chassis_link">
       <inertial>

Commit message: Rebase from 'upstream'

File: cob_description/urdf/cob4_base/base.urdf.xacro (robot description, xacro)
@@ -11,5 +11,5 @@
   <xacro:macro name="base" params="name tricycle_mode:=false forward:=true">
     <xacro:property name="drive_vel" value="19.95" />
-    <xacro:property name="steer_vel" value="117.81" />
+    <xacro:property name="steer_vel" value="12.00" /> <!-- Controller: 10.0, Driver: 12.0, Elmo: 15.0 -->
     <xacro:if value="${tricycle_mode}">
       <link name="${name}_pivot_link"/>
