Commit message: Rebase from 'release/kinetic/cob_description'

File: urdf/cob4_head/head.urdf.xacro (robot description, xacro)
@@ -1,10 +1,42 @@
 <?xml version="1.0"?>
 <robot xmlns:xacro="http://www.ros.org/wiki/xacro">
-  <xacro:include filename="$(find cob_description)/urdf/cob4_head/head.gazebo.xacro" />
-  <xacro:include filename="$(find cob_description)/urdf/cob4_head/head.transmission.xacro" />
+  <xacro:include filename="$(find cob_description)/urdf/common.xacro" />
+  <xacro:include filename="$(find cob_description)/urdf/cob4_head/head.gazebo.xacro"/>
+  <xacro:include filename="$(find cob_description)/urdf/cob4_head/head.transmission.xacro"/>
+  <!-- torso_2_joint is on the right side of the robot (different from CAD) -->
   <xacro:macro name="head" params="parent name *origin dof1:=false dof2:=false dof3:=false">
+    <xacro:property name="origin_1_joint">
+      <origin xyz="0 0 0.0305" rpy="0 0 0"/>
+    </xacro:property>
+    <xacro:property name="origin_2_joint">
+      <origin xyz="0 -0.07725 0.00439" rpy="0.349 0 0"/>
+    </xacro:property>
+    <xacro:property name="origin_3_joint">
+      <origin xyz="0 0.09849 0.04476" rpy="-0.349 0 0"/>
+    </xacro:property>
+    <xacro:head_template name="${name}" parent="${parent}" dof1="${dof1}" dof2="${dof2}" dof3="${dof3}">
+      <xacro:insert_block name="origin"/>
+    </xacro:head_template>
+  </xacro:macro>
+  <!-- torso_2_joint is on the left side of the robot (same as in CAD) -->
+  <xacro:macro name="head_cad" params="parent name *origin dof1:=false dof2:=false dof3:=false">
+    <xacro:property name="origin_1_joint">
+      <origin xyz="0 0 0.0305" rpy="0 0 0"/>
+    </xacro:property>
+    <xacro:property name="origin_2_joint">
+      <origin xyz="0 0.07725 0.00439" rpy="0.349 0 ${M_PI}"/>
+    </xacro:property>
+    <xacro:property name="origin_3_joint">
+      <origin xyz="0 0.09849 0.04476" rpy="0.349 0 -${M_PI}"/>
+    </xacro:property>
+    <xacro:head_template name="${name}" parent="${parent}" dof1="${dof1}" dof2="${dof2}" dof3="${dof3}">
+      <xacro:insert_block name="origin"/>
+    </xacro:head_template>
+  </xacro:macro>
+  <!-- configurable template -->
+  <xacro:macro name="head_template" params="parent name *origin dof1:=false dof2:=false dof3:=false">
     <joint name="${name}_base_joint" type="fixed">
-      <xacro:insert_block name="origin" />
-      <child link="${name}_base_link" />
+      <xacro:insert_block name="origin"/>
+      <child link="${name}_base_link"/>
       <parent link="${parent}"/>
     </joint>
@@ -12,13 +44,13 @@
       <xacro:default_inertial/>
       <visual>
-        <origin xyz="0 0 0" rpy="0 0 0" />
+        <origin xyz="0 0 0" rpy="0 0 0"/>
         <geometry>
-          <box size="0.001 0.001 0.001" />
+          <box size="0.001 0.001 0.001"/>
         </geometry>
       </visual>
       <collision>
-        <origin xyz="0 0 0" rpy="0 0 0" />
+        <origin xyz="0 0 0" rpy="0 0 0"/>
         <geometry>
-          <box size="0.001 0.001 0.001" />
+          <box size="0.001 0.001 0.001"/>
         </geometry>
       </collision>
@@ -26,15 +58,15 @@
     <xacro:unless value="${dof1}">
       <joint name="${name}_1_joint" type="fixed">
-        <origin xyz="0 0 0.0305" rpy="0 0 0"/>
+        <xacro:insert_block name="origin_1_joint"/>
         <parent link="${name}_base_link"/>
-        <child link="${name}_1_link" />
+        <child link="${name}_1_link"/>
       </joint>
     </xacro:unless>
     <xacro:if value="${dof1}">
       <joint name="${name}_1_joint" type="revolute">
-        <origin xyz="0 0 0.0305" rpy="0 0 0"/>
+        <xacro:insert_block name="origin_1_joint"/>
         <parent link="${name}_base_link"/>
-        <child link="${name}_1_link" />
-        <axis xyz="0 0 1" />
+        <child link="${name}_1_link"/>
+        <axis xyz="0 0 1"/>
         <limit effort="100" lower="-6.2831" upper="6.2831" velocity="1.4"/>
       </joint>
@@ -43,13 +75,13 @@
       <xacro:default_inertial/>
       <visual>
-        <origin xyz="0 0 0" rpy="0 0 0" />
+        <origin xyz="0 0 0" rpy="0 0 0"/>
         <geometry>
-          <box size="0.001 0.001 0.001" />
+          <box size="0.001 0.001 0.001"/>
         </geometry>
       </visual>
       <collision>
-        <origin xyz="0 0 0" rpy="0 0 0" />
+        <origin xyz="0 0 0" rpy="0 0 0"/>
         <geometry>
-          <box size="0.001 0.001 0.001" />
+          <box size="0.001 0.001 0.001"/>
         </geometry>
       </collision>
@@ -57,15 +89,15 @@
     <xacro:unless value="${dof2}">
       <joint name="${name}_2_joint" type="fixed">
-        <origin xyz="0 -0.07725 0.00439" rpy="0.349 0 0" />
+        <xacro:insert_block name="origin_2_joint"/>
         <parent link="${name}_1_link"/>
-        <child link="${name}_2_link" />
+        <child link="${name}_2_link"/>
       </joint>
     </xacro:unless>
     <xacro:if value="${dof2}">
       <joint name="${name}_2_joint" type="revolute">
-        <origin xyz="0 -0.07725 0.00439" rpy="0.349 0 0" />
+        <xacro:insert_block name="origin_2_joint"/>
         <parent link="${name}_1_link"/>
-        <child link="${name}_2_link" />
-        <axis xyz="0 0 1" />
+        <child link="${name}_2_link"/>
+        <axis xyz="0 0 1"/>
         <limit effort="100" lower="-6.2831" upper="6.2831" velocity="1.4"/>
       </joint>
@@ -74,13 +106,13 @@
       <xacro:default_inertial/>
       <visual>
-        <origin xyz="0 0 0" rpy="0 0 0" />
+        <origin xyz="0 0 0" rpy="0 0 0"/>
         <geometry>
-          <box size="0.001 0.001 0.001" />
+          <box size="0.001 0.001 0.001"/>
         </geometry>
       </visual>
       <collision>
-        <origin xyz="0 0 0" rpy="0 0 0" />
+        <origin xyz="0 0 0" rpy="0 0 0"/>
         <geometry>
-          <box size="0.001 0.001 0.001" />
+          <box size="0.001 0.001 0.001"/>
         </geometry>
       </collision>
@@ -88,15 +120,15 @@
     <xacro:unless value="${dof3}">
       <joint name="${name}_3_joint" type="fixed">
-        <origin xyz="0 0.09849 0.04476" rpy="-0.349 0 0" />
+        <xacro:insert_block name="origin_3_joint"/>
         <parent link="${name}_2_link"/>
-        <child link="${name}_3_link" />
+        <child link="${name}_3_link"/>
       </joint>
     </xacro:unless>
     <xacro:if value="${dof3}">
       <joint name="${name}_3_joint" type="revolute">
-        <origin xyz="0 0.09849 0.04476" rpy="-0.349 0 0" />
+        <xacro:insert_block name="origin_3_joint"/>
         <parent link="${name}_2_link"/>
-        <child link="${name}_3_link" />
-        <axis xyz="0 0 1" />
+        <child link="${name}_3_link"/>
+        <axis xyz="0 0 1"/>
         <limit effort="100" lower="-6.2831" upper="6.2831" velocity="1.4"/>
       </joint>
@@ -105,5 +137,5 @@
       <xacro:default_inertial/>
       <visual>
-        <origin xyz="0 0 0" rpy="0 0 0" />
+        <origin xyz="0 0 0" rpy="0 0 0"/>
         <geometry>
           <mesh filename="package://cob_description/meshes/cob4_head/head_link.dae"/>
@@ -111,5 +143,5 @@
       </visual>
       <collision>
-        <origin xyz="0 0 0" rpy="0 0 0" />
+        <origin xyz="0 0 0" rpy="0 0 0"/>
         <geometry>
           <mesh filename="package://cob_description/meshes/cob4_head/head_link_collision.stl"/>
@@ -118,12 +150,12 @@
     </link>
     <joint name="${name}_center_joint" type="fixed">
-      <origin xyz="0.0 0.0 -0.28247" rpy="0 0 0" />
+      <origin xyz="0.0 0.0 -0.28247" rpy="0 0 0"/>
       <parent link="${name}_3_link"/>
-      <child link="${name}_center_link" />
+      <child link="${name}_center_link"/>
     </joint>
     <link name="${name}_center_link"/>
     <!-- extensions -->
-    <xacro:head_gazebo name="${name}" />
-    <xacro:head_transmission name="${name}" dof1="${dof1}" dof2="${dof2}" dof3="${dof3}" />
+    <xacro:head_gazebo name="${name}"/>
+    <xacro:head_transmission name="${name}" dof1="${dof1}" dof2="${dof2}" dof3="${dof3}"/>
     <!-- ros_control plugin -->
     <xacro:if value="${(dof1 == True) or (dof2 == True) or (dof3 == True)}">

File: urdf/cob4_sensorring/sensorring.urdf.xacro (robot description, xacro)
@@ -1,4 +1,5 @@
 <?xml version="1.0"?>
 <robot xmlns:xacro="http://www.ros.org/wiki/xacro">
+  <xacro:include filename="$(find cob_description)/urdf/common.xacro" />
   <xacro:include filename="$(find cob_description)/urdf/cob4_sensorring/sensorring.gazebo.xacro" />
   <xacro:include filename="$(find cob_description)/urdf/cob4_sensorring/sensorring.transmission.xacro" />

File: urdf/cob4_torso/torso.urdf.xacro (robot description, xacro)
@@ -1,4 +1,5 @@
 <?xml version="1.0"?>
 <robot xmlns:xacro="http://www.ros.org/wiki/xacro">
+  <xacro:include filename="$(find cob_description)/urdf/common.xacro" />
   <xacro:include filename="$(find cob_description)/urdf/cob4_torso/torso.gazebo.xacro" />
   <xacro:include filename="$(find cob_description)/urdf/cob4_torso/torso.transmission.xacro" />

File: urdf/sensors/kinect.urdf.xacro (robot description, xacro)
@@ -1,4 +1,5 @@
 <?xml version="1.0"?>
 <root xmlns:xacro="http://www.ros.org/wiki/xacro">
+  <xacro:include filename="$(find cob_description)/urdf/common.xacro" />
   <xacro:include filename="$(find cob_description)/urdf/sensors/kinect.gazebo.xacro" />
   <xacro:macro name="cob_kinect_v0" params="name parent *origin ros_topic update_rate:=20 data_skip:=0 height:=480 width:=640">

File: urdf/sensors/prosilica.urdf.xacro (robot description, xacro)
@@ -2,4 +2,5 @@
 <robot xmlns:xacro="http://www.ros.org/wiki/xacro"
        name="LaserBlock">
+  <xacro:include filename="$(find cob_description)/urdf/common.xacro" />
   <xacro:include filename="$(find cob_description)/urdf/sensors/prosilica.gazebo.xacro" />
   <xacro:macro name="cob_prosilica_v0" params="name parent *origin ros_topic">

File: urdf/sensors/realsense.urdf.xacro (robot description, xacro)
@@ -1,4 +1,5 @@
 <?xml version="1.0"?>
 <robot xmlns:xacro="http://www.ros.org/wiki/xacro">
+  <xacro:include filename="$(find cob_description)/urdf/common.xacro" />
   <xacro:include filename="$(find cob_description)/urdf/sensors/realsense.gazebo.xacro" />
   <xacro:macro name="realsense" params="name parent ros_topic *origin">

File: urdf/sensors/realsense_d435.urdf.xacro (robot description, xacro)
@@ -1,4 +1,5 @@
 <?xml version="1.0"?>
 <robot xmlns:xacro="http://www.ros.org/wiki/xacro">
+  <xacro:include filename="$(find cob_description)/urdf/common.xacro" />
   <xacro:include filename="$(find cob_description)/urdf/sensors/realsense_d435.gazebo.xacro" />
   <xacro:macro name="realsense_d435" params="name parent *origin">

File: urdf/sensors/realsense_zr300.urdf.xacro (robot description, xacro)
@@ -1,4 +1,5 @@
 <?xml version="1.0"?>
 <robot xmlns:xacro="http://www.ros.org/wiki/xacro">
+  <xacro:include filename="$(find cob_description)/urdf/common.xacro" />
   <xacro:include filename="$(find cob_description)/urdf/sensors/realsense_zr300.gazebo.xacro" />
   <xacro:macro name="realsense_zr300" params="name parent ros_topic *origin">

File: urdf/sensors/rplidar.urdf.xacro (robot description, xacro)
@@ -1,4 +1,5 @@
 <?xml version="1.0"?>
 <robot xmlns:xacro="http://www.ros.org/wiki/xacro">
+  <xacro:include filename="$(find cob_description)/urdf/common.xacro" />
   <xacro:include filename="$(find cob_description)/urdf/sensors/rplidar.gazebo.xacro" />
   <xacro:property name="cylinder_radius" value="0.08" />

File: urdf/sensors/usb_cam.urdf.xacro (robot description, xacro)
@@ -2,4 +2,5 @@
 <robot xmlns:xacro="http://www.ros.org/wiki/xacro">
   <!-- This is a ELP-USBFHD01M-L21 or very similar board-level camera -->
+  <xacro:include filename="$(find cob_description)/urdf/common.xacro" />
   <xacro:include filename="$(find cob_description)/urdf/sensors/usb_cam.gazebo.xacro" />
   <xacro:macro name="usb_cam" params="name parent *origin ros_topic update_rate height width">
